File: Peavey_5150.sch (KiCad schematic (older format))
At the start: 315 parts, among them J1 INPUT, J10 INPUT, J165 SEND, J166 RETURN, J2 Power, J3 OUTPUT, J4 SWIM, J5 FOOTSWITCH, J6 KF2510, J7 KF2510, J8 KF2510, J9 KF2510, K1 G5V1, K2 G5V1, K3 G5V-2, K4 G5V1, K5 G5V1, Q1 IRF840, Q2 BC847, Q3 BC847, Q4 BC847, SW1 Ultra, SW2 Clean, SW3 Crunch, SW4 FX_loop, U1 MP4462, U2 AMS1117-3.3, U3 STM8S003F3P, U4 TLP222A

Commit message: Working on schematic
Parts:
- removed C1, C56, C57, C58, C6: .022uF/400V, symbol simple:C_US
- removed C10, C155: 0.033uF, symbol simple:C_US
- removed C13: .022uF, symbol simple:C_US
- removed C15: .1uF/250V, symbol simple:C_US
- removed C150: 100pF, symbol simple:C_US
- removed C151, C152, C17, C51: 470pF, symbol simple:C_US
- removed C153: 33uF/400V, symbol simple:C_US
- removed C154, C156: 0.022uF, symbol simple:C_US
- removed C157: 0.33uF, symbol simple:C_US
- removed C165: .22uF/400V, symbol simple:C_US
- removed C166: 2.2uF, symbol Device:CP1
- removed C167: 820pF, symbol simple:C_US
- removed C19, C48: 0.001uF, symbol simple:C_US
- removed C2: .001uF/630V, symbol simple:C_US
- removed C20: 39pF, symbol simple:C_US
- removed C27, C63: .068uF, symbol simple:C_US
- removed C3, C4, C5: 1uF/50V, symbol simple:C_US
- removed C31: 22uF, symbol Device:CP1
- removed J1, J10: INPUT, symbol simple:Jack_6.35
- removed J6, J7, J8, J9: KF2510, symbol Connector_Generic:Conn_01x04
- removed JP5: PLS-2, symbol Device:Jumper_NC_Small
- removed K1, K2, K4, K5: G5V1, symbol Relays:G5V1
- removed K?: G5V-2, symbol Relays:G5V-2
- removed R1, R101, R171, R3, R86: 100K, symbol Device:R_US
- removed R102, R155, R158, R93: 2.2K, symbol Device:R_US
- removed R11: 330K, symbol Device:R_US
- removed R12, R13, R157, R17: 82K, symbol Device:R_US
- removed R15: 39K, symbol Device:R_US
- removed R150, R170, R172, R4, R7, R96: 220K, symbol Device:R_US
- removed R151, R163: 33K, symbol Device:R_US
- removed R152, R154, R164, R19, R6, R82, R89: 470K, symbol Device:R_US
- removed R153: 18K, symbol Device:R_US
- removed R156, R27: 10K, symbol Device:R_US
- removed R159, R176, R25, R32, R40, R41, R87, R88, R9, R91: 1M, symbol Device:R_US
- removed R174, R75: 22K, symbol Device:R_US
- removed R175, R22: 68K, symbol Device:R_US
- removed R2: 210K, symbol Device:R_US
- removed R23: 6.8K, symbol Device:R_US
- removed R37: 10K 1W, symbol Device:R_US
- removed R63: 47R1W, symbol Device:R_US
- removed unit 1 of V1
- removed unit 2 of V1
- removed unit 1 of V2
- removed unit 2 of V2
- removed unit 2 of V5
- removed unit 1 of V5
- removed V6: (no value), Valve:Valve_Noval_P, symbol Valve:ECC83
- removed VR1, VR2, VR5: 1M, symbol simple:R_POT_US_P
- removed VR3: 25K, symbol simple:R_POT_US_P
- removed VR4: 250K, symbol simple:R_POT_US_P
- added unit 1 of K1
- added unit 1 of K2
- added unit 3 of K2
- added unit 1 of K4
- R24: value 47K -> 33K
- R94: value 33K -> 47K
- S1C1: renamed from SW?; value SW_SPDT -> (none)
- gave numbers to parts that had none: 67
- renumbered C26 to C31, R18 to R37, R20 to R63, R21 to R65, R29 to R66, R30 to R67, R43 to R68, VR7 to VR3, VR8 to VR4, VR9 to VR5, VR10 to VR7
Connections:
- net labels removed: C153_2, C153_2_TOP, GND_V3, GND_V3_TOP, K2B_1, K2B_1_TOP, K5A_2, K5A_2_TOP, K5A_9, K5A_9_TOP, ToneStack, V3+, V6A_7, V6A_7_TOP, С27, С27_TOP
- wire segments 1049 -> 730
Other:
- note added: "BRIGHT"
- note added: "CLEAN PRE"
- note added: "CLEAN VOL"
- note added: "ULTRA PRE"
- note added: "ULTRA VOL"
- note removed: "CRUNCH"
- note removed: "Vol"
- moved on the sheet: C11, C14, C158, C18, C37, C49, C52, C53, C59, C65, D7, J165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

Commit message: finish
Parts:
- removed S1C1: (no value), symbol Switch:SW_SPDT
- added K5: G5V1, symbol Relays:G5V1
Connections:
- net at D8.1 (K), K4.1, R49.1: now also K5.2
- net at D8.2 (A), K4.16, Q3.3 (C): now also K5.9
- net at C27.1, K4.13, K4.9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: now also K5.5, K5.6
- net at C10.2, R75.1: now also K5.10
- net CRUNCH_B renamed BRIGHT_B
- net CRUNCH_CLEAN renamed BRIGHT
- net CRUNCH_LED renamed BRIGHT_LED
Other:
- moved on the sheet: C10
Changed lines of the file:
@@
 	24950 16300 24950 16200
 Text Label 24450 15800 2    50   ~ 0
-CRUNCH_CLEAN
+BRIGHT
 Wire Wire Line
 	24550 15800 24450 15800
@@
 DIST_CLEAN
 Text Label 19450 15300 0    50   ~ 0
-CRUNCH_CLEAN
+BRIGHT
 Wire Wire Line
 	19350 15200 19450 15200
@@
 CLEAN_B
 Text Label 25650 18000 2    50   ~ 0
-CRUNCH_B
+BRIGHT_B
 Wire Wire Line
 	27500 18000 27400 18000
@@
 CLEAN_B
 Text Label 18050 15200 2    50   ~ 0
-CRUNCH_B
+BRIGHT_B
 Text Label 18050 15300 2    50   ~ 0
 ULTRA_B
@@
 CLEAN_LED
 Text Label 26450 17500 0    50   ~ 0
-CRUNCH_LED
+BRIGHT_LED
 Text Label 18050 15500 2    50   ~ 0
-CRUNCH_LED
+BRIGHT_LED
 Wire Wire Line
 	18150 15500 18050 15500
@@
 	27300 5700 26800 5700
 Connection ~ 27300 4950
-Connection ~ 7750 2600
 Wire Wire Line
-	7750 3100 7750 2600
+	7850 2600 7850 2500
 Wire Wire Line
-	7750 2600 7750 2500
+	7850 1900 7850 1500
+Connection ~ 7850 1900
+Connection ~ 7850 2100
 Wire Wire Line
-	7750 1900 7750 1500
-Connection ~ 7750 1900
-Connection ~ 7750 2100
+	7850 2100 7850 1900
 Wire Wire Line
-	7750 2100 7750 1900
-Wire Wire Line
-	7750 2100 7750 2200
+	7850 2100 7850 2200
 Connection ~ 6100 3850
 Wire Wire Line
@@
 Wire Wire Line
 	7150 3600 7050 3600
-Connection ~ 7050 3200
-Wire Wire Line
-	7050 3200 7050 3600
 $Comp
 L simple:C_US C27
@@
 $EndComp
 Connection ~ 7050 2850
+NoConn ~ 7750 3250
 Wire Wire Line
-	7050 3200 7050 2850
-Wire Wire Line
-	7250 3200 7050 3200
-NoConn ~ 7650 3300
-Wire Wire Line
-	7650 3100 7750 3100
-$Comp
-L Switch:SW_SPDT S1C1
-U 1 1 614C9514
-P 7450 3200
-F 0 "S1C1" H 7450 3000 50  0000 C CNN
-F 1 " " H 7450 2966 50  0000 C CNN
-F 2 "" H 7450 3200 50  0001 C CNN
-F 3 "~" H 7450 3200 50  0001 C CNN
-	1    7450 3200
-	1    0    0    1
-$EndComp
-Wire Wire Line
-	7450 2600 7750 2600
+	7450 2600 7850 2600
 Wire Wire Line
 	7150 2600 7050 2600
@@
 	6350 1900 6450 1900
 Wire Wire Line
-	7650 1900 7750 1900
+	7650 1900 7850 1900
 Wire Wire Line
-	7750 1500 7650 1500
+	7850 1500 7650 1500
 $Comp
 L simple:C_US C13
@@
 $EndComp
 Wire Wire Line
-	7050 2100 7750 2100
+	7050 2100 7850 2100
 $Comp
 L simple:C_US C10
 U 1 1 60EB3129
-P 7750 2350
-F 0 "C10" H 7650 2400 50  0000 R CNN
-F 1 "470pF" H 7650 2250 50  0000 R CNN
-F 2 "" H 7750 2350 50  0001 C CNN
-F 3 "" H 7750 2350 50  0001 C CNN
-	1    7750 2350
+P 7850 2350
+F 0 "C10" H 7750 2400 50  0000 R CNN
+F 1 "470pF" H 7750 2250 50  0000 R CNN
+F 2 "" H 7850 2350 50  0001 C CNN
+F 3 "" H 7850 2350 50  0001 C CNN
+	1    7850 2350
 	1    0    0    -1
 $EndComp
@@
 Wire Wire Line
 	17350 3100 17350 3550
-Text Notes 7750 3250 0    50   ~ 0
+Text Notes 7900 3200 0    50   ~ 0
 BRIGHT
 Text Label 6400 15300 0    50   ~ 0
@@
 	0    -1   -1   0
 $EndComp
+$Comp
+L Relays:G5V1 K5
+U 2 1 5ED8EB44
+P 7500 3150
+F 0 "K5" H 7450 2869 50  0000 C CNN
+F 1 "G5V1" H 7450 2960 50  0000 C CNN
+F 2 "" H 7500 3150 50  0001 C CNN
+F 3 "" H 7500 3150 50  0001 C CNN
+	2    7500 3150
+	1    0    0    1
+$EndComp
+Wire Wire Line
+	7050 2850 7050 3050
+Wire Wire Line
+	7750 3050 7850 3050
+Wire Wire Line
+	7850 3050 7850 2600
+Connection ~ 7850 2600
+Wire Wire Line
+	7150 3050 7050 3050
+Connection ~ 7050 3050
+Wire Wire Line
+	7050 3050 7050 3150
+Wire Wire Line
+	7150 3150 7050 3150
+Connection ~ 7050 3150
+Wire Wire Line
+	7050 3150 7050 3600
+$Comp
+L Relays:G5V1 K5
+U 1 1 5F003346
+P 25800 15100
+F 0 "K5" H 25645 15146 50  0000 R CNN
+F 1 "G5V1" H 25645 15055 50  0000 R CNN
+F 2 "" H 25800 15100 50  0001 C CNN
+F 3 "" H 25800 15100 50  0001 C CNN
+	1    25800 15100
+	-1   0    0    -1
+$EndComp
+Wire Wire Line
+	25800 14800 25800 14700
+Wire Wire Line
+	25800 14700 25350 14700
+Wire Wire Line
+	25800 15400 25800 15500
+Wire Wire Line
+	25800 15500 25350 15500
 $EndSCHEMATC

Commit message: add led
Parts:
- removed C44: 0.1uF, symbol simple:C_US
- removed D3: WHITE, symbol Device:LED
- removed D5: RED, symbol Device:LED
- removed R60: 1K, symbol Device:R_US
- removed SW1: Ultra, symbol Switch:SW_Push
- added D3: LED_Dual_AACC, symbol Device:LED_Dual_AACC
- R56: value 47K -> 1K
Connections:
- net +3V3: no longer R56.2
- net GND: now also D3.3 (K1), D3.4 (K2)
- net at R58.1: now also D3.2 (A2)
- net ULTRA_B: no longer names the net of R56.1
- net ULTRA_B: now also D3.1 (A1); no longer U3.15 (PC5)
- new net ULTRA_LED: R56.2, U3.15 (PC5)
Other:
- moved on the sheet: C43, D4, R55, R58, R59, SW3

Commit message: Some values fixed
Parts:
- added R?: 10K, symbol Device:R_US
- C1, C2, C52, C56, C57, C58, C6: value .022uF/400V -> .022uF 400V
- C11: value 047A400 -> 0.047uF 450V
- C14: value 470pF -> 470pF 50v
- C15: value .1uF/250V -> .1uF 250V
- C158: value 0.0047uF -> 0.0047uF 50v
- C18, C37: value 0.022uF -> 0.022uF 50v
- C20: value 39pF -> 39pF 50V
- C26: value 22 -> 22uF
- C3, C4, C5: value 1uF/50V -> 1uF 50V
- C49: value 022R400 -> .022uF 400V
- C53, C65: value 33R400 -> 0.33uF 400v
- C59: value 0.1uF -> 0.01uF 50v
- R103, R33, R86: value 100K -> 100K 1/4W
- R12: value 1.82K -> 1.82K 1/4W
- R14: value 3.3K -> 3.3K 1/4W
- R160, R161, R25, R26, R79: value 1M -> 1M 1/4W
- R2, R4, R85, R96: value 220K -> 220K 1/4W
- R20: value 470K -> 220K
- R22: value 68K -> 68K 1/4W
- R27, R30: value 22K -> 22K 1/4W
- R5: value 68KP1 -> 68K 1/4W
- R62, R64: value 220KW1 -> 220K 1W
- R80: value 1K -> 1K 1/4W
- R81: value 2.2M -> 2.2M 1/4W
Connections:
- net at C18.1, C37.1: now also R?.1; no longer VR12.1
- new net: R?.2, VR12.1
Other:
- moved on the sheet: C11, C14, C49, C53, C59, C65, J165, J166, J3, K3B, K3C, R1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

Commit message: Input changes
Parts:
- removed R27: 22K 1/4W, symbol Device:R_US
- C1, C10, C11, C12, C13, C14, C15, C158, C16, C17, C18, C19, C2, C20, C22, C24, C25, C27, C3, C31, C32, C35, C36, C37, C39, C4, C40, C41, C42, C43, C45, C48, C49, C5, C51, C52, C53, C56, C57, C58, C59, C6, C63, C65, C7, C8, C9: symbol simple:C_US -> Peavey_5150-rescue:C_US-simple
- F1, F2: symbol simple:Fuse -> Peavey_5150-rescue:Fuse-simple
- J165, J166, J3, J5: symbol simple:Jack_6.35 -> Peavey_5150-rescue:Jack_6.35-simple
- J37: value INPUT -> INPUT FRONT; symbol simple:Jack_6.35 -> Peavey_5150-rescue:Jack_6.35-simple
- J39: value INPUT -> INPUT REAR; symbol simple:Jack_6.35 -> Peavey_5150-rescue:Jack_6.35-simple
- K1, K2, K3, K4: symbol Relays:G5V-2 -> Peavey_5150-rescue:G5V-2-Relays
- K5: symbol Relays:G5V1 -> Peavey_5150-rescue:G5V1-Relays
- U1: symbol simple:MP4462 -> Peavey_5150-rescue:MP4462-simple
- VR1, VR11, VR12, VR13, VR2, VR3, VR4, VR5, VR6, VR7: symbol simple:R_POT_US_P -> Peavey_5150-rescue:R_POT_US_P-simple
Connections:
- net Earth: now also J39.2; no longer J37.2
- net at J37.1: now also R22.1, R25.1; no longer J39.2
- new net: C15.1, J37.2
Other:
- moved on the sheet: C15

Commit message: Update
Parts:
- SW3: value Crunch -> Bright
- gave numbers to parts that had none: 1
Changed lines of the file:
@@
 P 27300 18250
 F 0 "SW3" V 27254 18398 50  0000 L CNN
-F 1 "Crunch" V 27345 18398 50  0000 L CNN
+F 1 "Bright" V 27345 18398 50  0000 L CNN
 F 2 "" H 27300 18450 50  0001 C CNN
 F 3 "~" H 27300 18450 50  0001 C CNN
@@
 Connection ~ 20200 3150
 $Comp
-L Device:R_US R?
+L Device:R_US R27
 U 1 1 5F020BC7
 P 20200 3800
-F 0 "R?" H 20400 3750 50  0000 R CNN
+F 0 "R27" H 20400 3750 50  0000 R CNN
 F 1 "10K" H 20400 3850 50  0000 R CNN
 F 2 "" V 20240 3790 50  0001 C CNN
