File: Peavey_5150.sch (KiCad schematic (older format))
At the start: 203 parts, among them J165 SEND, J166 RETURN, J2 Power, J3 OUTPUT, J37 INPUT FRONT, J39 INPUT REAR, J4 SWIM, J5 FOOTSWITCH, K1 G5V-2, K2 G5V-2, K3 G5V-2, K4 G5V-2, K5 G5V1, Q1 IRF840, Q2 BC847, Q3 BC847, Q4 BC847, SW2 Clean, SW3 Bright, SW4 FX_loop, U1 MP4462, U2 AMS1117-3.3, U3 STM8S003F3P, U4 TLP222A

Commit message: Footprint partial assignment
Parts:
- removed D3: LED_Dual_AACC, symbol Device:LED_Dual_AACC
- removed D4: WHITE, symbol Device:LED
- removed R59: 1K, symbol Device:R_US
- added D3: GREEN, LED_SMD:LED_0603_1608Metric, symbol Device:LED
- added D5: RED, LED_SMD:LED_0603_1608Metric, symbol Device:LED
- added K?: G5V1, symbol Peavey_5150-rescue:G5V1-Relays-Peavey_5150-rescue
- C1, C2, C49, C56, C57, C58, C6: footprint (none) -> Peavey-EVH5150:C_UNIVERSAL
- C3, C4, C5: footprint (none) -> Peavey-EVH5150:CP_UNIVERSAL
- CR1, CR2, CR3, CR4: footprint Diode_THT:D_DO-41_SOD81_P10.16mm_Horizontal -> Diode_SMD:D_SMC
- D6: value WHITE -> RED; footprint (none) -> LED_SMD:LED_0603_1608Metric
- J2: footprint (none) -> Peavey-EVH5150:X977T08
- J4: footprint (none) -> Connector_PinHeader_2.54mm:PinHeader_1x03_P2.54mm_Vertical
Connections:
- wire segments 723 -> 720
- no-connect marks 8 -> 9
Changed lines of the file:
@@
 EESchema Schematic File Version 4
-LIBS:Peavey_5150-cache
-EELAYER 29 0
+EELAYER 30 0
 EELAYER END
 $Descr A1 33110 23386
@@
 F 0 "CR1" V 6654 17079 50  0000 L CNN
 F 1 "S3M" V 6745 17079 50  0000 L CNN
-F 2 "Diode_THT:D_DO-41_SOD81_P10.16mm_Horizontal" H 6700 16825 50  0001 C CNN
+F 2 "Diode_SMD:D_SMC" H 6700 16825 50  0001 C CNN
 F 3 "http://www.vishay.com/docs/88503/1n4001.pdf" H 6700 17000 50  0001 C CNN
 	1    6700 17000
@@
 F 0 "CR3" V 7296 16921 50  0000 R CNN
 F 1 "S3M" V 7205 16921 50  0000 R CNN
-F 2 "Diode_THT:D_DO-41_SOD81_P10.16mm_Horizontal" H 7250 16825 50  0001 C CNN
+F 2 "Diode_SMD:D_SMC" H 7250 16825 50  0001 C CNN
 F 3 "http://www.vishay.com/docs/88503/1n4001.pdf" H 7250 17000 50  0001 C CNN
 	1    7250 17000
@@
 F 0 "CR2" V 6746 17421 50  0000 R CNN
 F 1 "S3M" V 6655 17421 50  0000 R CNN
-F 2 "Diode_THT:D_DO-41_SOD81_P10.16mm_Horizontal" H 6700 17325 50  0001 C CNN
+F 2 "Diode_SMD:D_SMC" H 6700 17325 50  0001 C CNN
 F 3 "http://www.vishay.com/docs/88503/1n4001.pdf" H 6700 17500 50  0001 C CNN
 	1    6700 17500
@@
 F 0 "CR4" V 7204 17579 50  0000 L CNN
 F 1 "S3M" V 7295 17579 50  0000 L CNN
-F 2 "Diode_THT:D_DO-41_SOD81_P10.16mm_Horizontal" H 7250 17325 50  0001 C CNN
+F 2 "Diode_SMD:D_SMC" H 7250 17325 50  0001 C CNN
 F 3 "http://www.vishay.com/docs/88503/1n4001.pdf" H 7250 17500 50  0001 C CNN
 	1    7250 17500
@@
 F 0 "J4" H 20880 14442 50  0000 L CNN
 F 1 "SWIM" H 20880 14351 50  0000 L CNN
-F 2 "" H 20800 14400 50  0001 C CNN
+F 2 "Connector_PinHeader_2.54mm:PinHeader_1x03_P2.54mm_Vertical" H 20800 14400 50  0001 C CNN
 F 3 "~" H 20800 14400 50  0001 C CNN
 	1    20800 14400
@@
 F 0 "J2" H 2168 14567 50  0000 C CNN
 F 1 "Power" H 2168 14476 50  0000 C CNN
-F 2 "" H 2250 14050 50  0001 C CNN
+F 2 "Peavey-EVH5150:X977T08" H 2250 14050 50  0001 C CNN
 F 3 "~" H 2250 14050 50  0001 C CNN
 	1    2250 14050
@@
 F 0 "C49" V 24700 5750 50  0000 L CNN
 F 1 ".022uF 400V" V 24400 5700 50  0000 L CNN
-F 2 "" H 24550 5850 50  0001 C CNN
+F 2 "Peavey-EVH5150:C_UNIVERSAL" H 24550 5850 50  0001 C CNN
 F 3 "" H 24550 5850 50  0001 C CNN
 	1    24550 5850
@@
 P 29950 18150
 F 0 "D6" V 29989 18032 50  0000 R CNN
-F 1 "WHITE" V 29898 18032 50  0000 R CNN
-F 2 "" H 29950 18150 50  0001 C CNN
+F 1 "RED" V 29898 18032 50  0000 R CNN
+F 2 "LED_SMD:LED_0603_1608Metric" H 29950 18150 50  0001 C CNN
 F 3 "~" H 29950 18150 50  0001 C CNN
 	1    29950 18150
@@
 	29950 18000 29950 17900
 $Comp
-L Device:R_US R59
-U 1 1 6229F78F
-P 27850 17700
-F 0 "R59" H 27800 17650 50  0000 R CNN
-F 1 "1K" H 27800 17750 50  0000 R CNN
-F 2 "" V 27890 17690 50  0001 C CNN
-F 3 "~" H 27850 17700 50  0001 C CNN
-	1    27850 17700
-	-1   0    0    1
-$EndComp
-Wire Wire Line
-	27850 17550 27850 17450
-$Comp
-L Device:LED D4
-U 1 1 6229F79B
-P 27850 18100
-F 0 "D4" V 27889 17982 50  0000 R CNN
-F 1 "WHITE" V 27798 17982 50  0000 R CNN
-F 2 "" H 27850 18100 50  0001 C CNN
-F 3 "~" H 27850 18100 50  0001 C CNN
-	1    27850 18100
-	0    -1   -1   0
-$EndComp
-$Comp
-L power:GND #PWR084
-U 1 1 6229F7A5
-P 27850 18650
-F 0 "#PWR084" H 27850 18400 50  0001 C CNN
-F 1 "GND" H 27855 18477 50  0000 C CNN
-F 2 "" H 27850 18650 50  0001 C CNN
-F 3 "" H 27850 18650 50  0001 C CNN
-	1    27850 18650
-	1    0    0    -1
-$EndComp
-Wire Wire Line
-	27850 18650 27850 18250
-Wire Wire Line
-	27850 17950 27850 17850
-$Comp
 L Device:R_US R58
 U 1 1 623C5EE6
@@
 $EndComp
 Wire Wire Line
-	25350 18000 25350 17900
+	25350 18150 25350 17900
 Text Label 19450 14900 0    50   ~ 0
 CLEAN_LED
@@
 Text Label 25350 17500 2    50   ~ 0
 CLEAN_LED
-Text Label 27850 17450 0    50   ~ 0
-BRIGHT_LED
 Text Label 18050 15500 2    50   ~ 0
 BRIGHT_LED
@@
 F 0 "C6" V 4750 2000 50  0000 C CNN
 F 1 ".022uF 400V" V 4450 2000 50  0000 C CNN
-F 2 "" H 4600 2000 50  0001 C CNN
+F 2 "Peavey-EVH5150:C_UNIVERSAL" H 4600 2000 50  0001 C CNN
 F 3 "" H 4600 2000 50  0001 C CNN
 	1    4600 2000
@@
 F 0 "C3" H 3650 3300 50  0000 R CNN
 F 1 "1uF 50V" H 3650 3150 50  0000 R CNN
-F 2 "" H 3750 3250 50  0001 C CNN
+F 2 "Peavey-EVH5150:CP_UNIVERSAL" H 3750 3250 50  0001 C CNN
 F 3 "" H 3750 3250 50  0001 C CNN
 	1    3750 3250
@@
 F 0 "C4" H 8900 3800 50  0000 R CNN
 F 1 "1uF 50V" H 8900 3650 50  0000 R CNN
-F 2 "" H 9000 3750 50  0001 C CNN
+F 2 "Peavey-EVH5150:CP_UNIVERSAL" H 9000 3750 50  0001 C CNN
 F 3 "" H 9000 3750 50  0001 C CNN
 	1    9000 3750
@@
 F 0 "C2" V 10000 2500 50  0000 C CNN
 F 1 ".022uF 400V" V 9700 2500 50  0000 C CNN
-F 2 "" H 9850 2500 50  0001 C CNN
+F 2 "Peavey-EVH5150:C_UNIVERSAL" H 9850 2500 50  0001 C CNN
 F 3 "" H 9850 2500 50  0001 C CNN
 	1    9850 2500
@@
 F 0 "C1" V 11750 2500 50  0000 C CNN
 F 1 ".022uF 400V" V 11450 2500 50  0000 C CNN
-F 2 "" H 11600 2500 50  0001 C CNN
+F 2 "Peavey-EVH5150:C_UNIVERSAL" H 11600 2500 50  0001 C CNN
 F 3 "" H 11600 2500 50  0001 C CNN
 	1    11600 2500
@@
 F 0 "C5" H 12700 3800 50  0000 R CNN
 F 1 "1uF 50V" H 12700 3650 50  0000 R CNN
-F 2 "" H 12800 3750 50  0001 C CNN
+F 2 "Peavey-EVH5150:CP_UNIVERSAL" H 12800 3750 50  0001 C CNN
 F 3 "" H 12800 3750 50  0001 C CNN
 	1    12800 3750
@@
 F 0 "C57" V 14050 2500 50  0000 C CNN
 F 1 ".022uF 400V" V 13750 2500 50  0000 C CNN
-F 2 "" H 13900 2500 50  0001 C CNN
+F 2 "Peavey-EVH5150:C_UNIVERSAL" H 13900 2500 50  0001 C CNN
 F 3 "" H 13900 2500 50  0001 C CNN
 	1    13900 2500
@@
 F 0 "C56" V 15800 2700 50  0000 C CNN
 F 1 ".022uF 400V" V 15500 2700 50  0000 C CNN
-F 2 "" H 15650 2700 50  0001 C CNN
+F 2 "Peavey-EVH5150:C_UNIVERSAL" H 15650 2700 50  0001 C CNN
 F 3 "" H 15650 2700 50  0001 C CNN
 	1    15650 2700
@@
 F 0 "C58" V 17200 2500 50  0000 C CNN
 F 1 ".022uF 400V" V 16900 2500 50  0000 C CNN
-F 2 "" H 17050 2500 50  0001 C CNN
+F 2 "Peavey-EVH5150:C_UNIVERSAL" H 17050 2500 50  0001 C CNN
 F 3 "" H 17050 2500 50  0001 C CNN
 	1    17050 2500
@@
 Wire Wire Line
 	25800 15500 25350 15500
-$Comp
-L Device:LED_Dual_AACC D3
-U 1 1 5F1E96D5
-P 25450 18300
-F 0 "D3" V 25404 18588 50  0000 L CNN
-F 1 "LED_Dual_AACC" V 25495 18588 50  0000 L CNN
-F 2 "" H 25480 18300 50  0001 C CNN
-F 3 "~" H 25480 18300 50  0001 C CNN
-	1    25450 18300
-	0    1    1    0
-$EndComp
 Wire Wire Line
-	25350 18700 25350 18600
+	25350 18700 25350 18450
 $Comp
 L Device:R_US R56
@@
 $EndComp
 Wire Wire Line
-	25550 18000 25550 17900
+	25550 18150 25550 17900
 $Comp
 L power:GND #PWR01
@@
 $EndComp
 Wire Wire Line
-	25550 18700 25550 18600
+	25550 18700 25550 18450
 Wire Wire Line
 	25550 17600 25550 17500
@@
 Wire Wire Line
 	6300 4450 7550 4450
+$Comp
+L Device:LED D5
+U 1 1 5FB8C65B
+P 25550 18300
+F 0 "D5" V 25589 18182 50  0000 R CNN
+F 1 "RED" V 25498 18182 50  0000 R CNN
+F 2 "LED_SMD:LED_0603_1608Metric" H 25550 18300 50  0001 C CNN
+F 3 "~" H 25550 18300 50  0001 C CNN
+	1    25550 18300
+	0    -1   -1   0
+$EndComp
+$Comp
+L Device:LED D3
+U 1 1 5FB8F770
+P 25350 18300
+F 0 "D3" V 25389 18182 50  0000 R CNN
+F 1 "GREEN" V 25298 18182 50  0000 R CNN
+F 2 "LED_SMD:LED_0603_1608Metric" H 25350 18300 50  0001 C CNN
+F 3 "~" H 25350 18300 50  0001 C CNN
+	1    25350 18300
+	0    1    -1   0
+$EndComp
+NoConn ~ 18050 15500
+$Comp
+L Peavey_5150-rescue:G5V1-Relays-Peavey_5150-rescue K?
+U 2 1 60063336
+P 8000 4800
+F 0 "K?" H 7950 4519 50  0000 C CNN
+F 1 "G5V1" H 7950 4610 50  0000 C CNN
+F 2 "" H 8000 4800 50  0001 C CNN
+F 3 "" H 8000 4800 50  0001 C CNN
+	2    8000 4800
+	1    0    0    1
+$EndComp
 $EndSCHEMATC

Commit message: Footprint update
Parts:
- gave numbers to parts that had none: 1
Changed lines of the file:
@@
 NoConn ~ 18050 15500
 $Comp
-L Peavey_5150-rescue:G5V1-Relays-Peavey_5150-rescue K?
+L Peavey_5150-rescue:G5V1-Relays-Peavey_5150-rescue K6
 U 2 1 60063336
 P 8000 4800
-F 0 "K?" H 7950 4519 50  0000 C CNN
+F 0 "K6" H 7950 4519 50  0000 C CNN
 F 1 "G5V1" H 7950 4610 50  0000 C CNN
 F 2 "" H 8000 4800 50  0001 C CNN

Commit message: add relays
Parts:
- removed K2: G5V-2, symbol Peavey_5150-rescue:G5V-2-Relays-Peavey_5150-rescue
- added K2: G5V1, Peavey-EVH5150:Relay_SPDT_Omron_G5V-1, symbol Peavey_5150-rescue:G5V1-Relays-Peavey_5150-rescue
- added unit 1 of K6
- K1, K3, K4: footprint (none) -> Peavey-EVH5150:Relay_DPDT_Omron_G5V-2
- K5, K6: footprint (none) -> Peavey-EVH5150:Relay_SPDT_Omron_G5V-1
Connections:
- net at C52.1, R81.2, U4.3: now also K6.5, K6.6
- net at VR7.3: now also K6.10
- net at D7.1 (K), K1.1, R46.1: now also K2.2, K6.2
- net at D7.2 (A), K1.16, Q2.3 (C): now also K2.9, K6.9
- net at K6.1: now also VR6.3
- net at C27.2, VR1.3: now also K2.1
- net at R82.1: now also K2.5, K2.6
- net at C19.2, R40.1, VR2.3: now also K2.10
Other:
- note added: "12V 12.5mA"
- note added: "12V 41.7mA"
- moved on the sheet: K1A, K6B
Changed lines of the file:
@@
 EESchema Schematic File Version 4
-EELAYER 30 0
+LIBS:Peavey_5150-cache
+EELAYER 29 0
 EELAYER END
 $Descr A1 33110 23386
@@
 	22900 3250 23000 3250
 Wire Wire Line
-	23800 3500 23800 3150
+	23800 3500 23800 3250
 $Comp
 L Peavey_5150-rescue:R_POT_US_P-simple-Peavey_5150-rescue VR12
@@
 F 0 "K3" H 26650 3750 50  0000 C CNN
 F 1 "G5V-2" H 26700 3500 50  0000 C CNN
-F 2 "" H 26900 3650 50  0001 C CNN
+F 2 "Peavey-EVH5150:Relay_DPDT_Omron_G5V-2" H 26900 3650 50  0001 C CNN
 F 3 "" H 26900 3650 50  0001 C CNN
 	2    26900 3650
@@
 F 0 "K3" H 27505 15146 50  0000 L CNN
 F 1 "G5V-2" H 27505 15055 50  0000 L CNN
-F 2 "" H 27350 15100 50  0001 C CNN
+F 2 "Peavey-EVH5150:Relay_DPDT_Omron_G5V-2" H 27350 15100 50  0001 C CNN
 F 3 "" H 27350 15100 50  0001 C CNN
 	1    27350 15100
@@
 F 0 "K3" H 26650 5900 50  0000 C CNN
 F 1 "G5V-2" H 26700 5650 50  0000 C CNN
-F 2 "" H 26900 5800 50  0001 C CNN
+F 2 "Peavey-EVH5150:Relay_DPDT_Omron_G5V-2" H 26900 5800 50  0001 C CNN
 F 3 "" H 26900 5800 50  0001 C CNN
 	3    26900 5800
@@
 	23150 14700 22800 14700
 Wire Wire Line
-	22800 14700 22800 14800
+	22250 14700 22250 14800
 Connection ~ 23150 14700
 Wire Wire Line
 	23150 14700 23150 14800
 Wire Wire Line
-	22800 15400 22800 15500
+	22250 15400 22250 15500
 Wire Wire Line
-	22800 15500 23150 15500
+	22250 15500 22800 15500
 Connection ~ 23150 15500
 Wire Wire Line
@@
 Wire Wire Line
 	7650 4000 7550 4000
-$Comp
-L Peavey_5150-rescue:G5V-2-Relays-Peavey_5150-rescue K2
-U 2 1 61BF8E8B
-P 7900 4100
-F 0 "K2" H 7650 4250 50  0000 C CNN
-F 1 "G5V-2" H 7700 4000 50  0000 C CNN
-F 2 "" H 7900 4100 50  0001 C CNN
-F 3 "" H 7900 4100 50  0001 C CNN
-	2    7900 4100
-	-1   0    0    -1
-$EndComp
 Wire Wire Line
 	7050 4250 7050 4150
@@
 F 0 "K4" H 6350 2750 50  0000 C CNN
 F 1 "G5V-2" H 6400 2500 50  0000 C CNN
-F 2 "" H 6600 2600 50  0001 C CNN
+F 2 "Peavey-EVH5150:Relay_DPDT_Omron_G5V-2" H 6600 2600 50  0001 C CNN
 F 3 "" H 6600 2600 50  0001 C CNN
 	3    6600 2600
@@
 F 0 "K4" H 5850 2100 50  0000 C CNN
 F 1 "G5V-2" H 5900 1850 50  0000 C CNN
-F 2 "" H 6100 2000 50  0001 C CNN
+F 2 "Peavey-EVH5150:Relay_DPDT_Omron_G5V-2" H 6100 2000 50  0001 C CNN
 F 3 "" H 6100 2000 50  0001 C CNN
 	2    6100 2000
@@
 F 0 "K1" H 10600 5150 50  0000 C CNN
 F 1 "G5V-2" H 10650 4900 50  0000 C CNN
-F 2 "" H 10850 5000 50  0001 C CNN
+F 2 "Peavey-EVH5150:Relay_DPDT_Omron_G5V-2" H 10850 5000 50  0001 C CNN
 F 3 "" H 10850 5000 50  0001 C CNN
 	2    10850 5000
@@
 F 0 "K1" H 10600 4700 50  0000 C CNN
 F 1 "G5V-2" H 10650 4450 50  0000 C CNN
-F 2 "" H 10850 4550 50  0001 C CNN
+F 2 "Peavey-EVH5150:Relay_DPDT_Omron_G5V-2" H 10850 4550 50  0001 C CNN
 F 3 "" H 10850 4550 50  0001 C CNN
 	3    10850 4550
@@
 GNDPWR
 $Comp
-L Peavey_5150-rescue:G5V-2-Relays-Peavey_5150-rescue K2
-U 1 1 6AA3417A
-P 23150 15100
-F 0 "K2" H 22900 15150 50  0000 C CNN
-F 1 "G5V-2" H 22850 15050 50  0000 C CNN
-F 2 "" H 23150 15100 50  0001 C CNN
-F 3 "" H 23150 15100 50  0001 C CNN
-	1    23150 15100
-	-1   0    0    -1
-$EndComp
-$Comp
 L Peavey_5150-rescue:G5V-2-Relays-Peavey_5150-rescue K1
 U 1 1 6AA3618E
-P 22800 15100
-F 0 "K1" H 23050 15150 50  0000 C CNN
-F 1 "G5V-2" H 23100 15050 50  0000 C CNN
-F 2 "" H 22800 15100 50  0001 C CNN
-F 3 "" H 22800 15100 50  0001 C CNN
-	1    22800 15100
+P 22250 15100
+F 0 "K1" H 22500 15150 50  0000 C CNN
+F 1 "G5V-2" H 22550 15050 50  0000 C CNN
+F 2 "Peavey-EVH5150:Relay_DPDT_Omron_G5V-2" H 22250 15100 50  0001 C CNN
+F 3 "" H 22250 15100 50  0001 C CNN
+	1    22250 15100
 	-1   0    0    -1
 $EndComp
@@
 F 0 "K4" H 25200 15150 50  0000 C CNN
 F 1 "G5V-2" H 25250 15050 50  0000 C CNN
-F 2 "" H 24950 15100 50  0001 C CNN
+F 2 "Peavey-EVH5150:Relay_DPDT_Omron_G5V-2" H 24950 15100 50  0001 C CNN
 F 3 "" H 24950 15100 50  0001 C CNN
 	1    24950 15100
 	-1   0    0    -1
 $EndComp
-$Comp
-L Peavey_5150-rescue:G5V-2-Relays-Peavey_5150-rescue K2
-U 3 1 6AC21A8E
-P 23250 3150
-F 0 "K2" H 23000 3300 50  0000 C CNN
-F 1 "G5V-2" H 23050 3050 50  0000 C CNN
-F 2 "" H 23250 3150 50  0001 C CNN
-F 3 "" H 23250 3150 50  0001 C CNN
-	3    23250 3150
-	-1   0    0    -1
-$EndComp
 Wire Wire Line
 	23600 3150 23800 3150
@@
 F 0 "K5" H 7450 2869 50  0000 C CNN
 F 1 "G5V1" H 7450 2960 50  0000 C CNN
-F 2 "" H 7500 3150 50  0001 C CNN
+F 2 "Peavey-EVH5150:Relay_SPDT_Omron_G5V-1" H 7500 3150 50  0001 C CNN
 F 3 "" H 7500 3150 50  0001 C CNN
 	2    7500 3150
@@
 F 0 "K5" H 25645 15146 50  0000 R CNN
 F 1 "G5V1" H 25645 15055 50  0000 R CNN
-F 2 "" H 25800 15100 50  0001 C CNN
+F 2 "Peavey-EVH5150:Relay_SPDT_Omron_G5V-1" H 25800 15100 50  0001 C CNN
 F 3 "" H 25800 15100 50  0001 C CNN
 	1    25800 15100
@@
 L Peavey_5150-rescue:G5V1-Relays-Peavey_5150-rescue K6
 U 2 1 60063336
-P 8000 4800
-F 0 "K6" H 7950 4519 50  0000 C CNN
-F 1 "G5V1" H 7950 4610 50  0000 C CNN
-F 2 "" H 8000 4800 50  0001 C CNN
-F 3 "" H 8000 4800 50  0001 C CNN
-	2    8000 4800
-	1    0    0    1
+P 23250 3150
+F 0 "K6" H 23150 3400 50  0000 C CNN
+F 1 "G5V1" H 23150 3300 50  0000 C CNN
+F 2 "Peavey-EVH5150:Relay_SPDT_Omron_G5V-1" H 23250 3150 50  0001 C CNN
+F 3 "" H 23250 3150 50  0001 C CNN
+	2    23250 3150
+	-1   0    0    -1
 $EndComp
+$Comp
+L Peavey_5150-rescue:G5V1-Relays-Peavey_5150-rescue K2
+U 2 1 5FB967F2
+P 7900 4100
+F 0 "K2" H 7800 4350 50  0000 C CNN
+F 1 "G5V1" H 7800 4250 50  0000 C CNN
+F 2 "Peavey-EVH5150:Relay_SPDT_Omron_G5V-1" H 7900 4100 50  0001 C CNN
+F 3 "" H 7900 4100 50  0001 C CNN
+	2    7900 4100
+	-1   0    0    -1
+$EndComp
+Wire Wire Line
+	8250 4200 8450 4200
+Wire Wire Line
+	8450 4200 8450 4100
+Connection ~ 8450 4100
+Wire Wire Line
+	23600 3250 23800 3250
+Connection ~ 23800 3250
+Wire Wire Line
+	23800 3250 23800 3150
+$Comp
+L Peavey_5150-rescue:G5V1-Relays-Peavey_5150-rescue K2
+U 1 1 5FCD7242
+P 22800 15100
+F 0 "K2" H 22645 15146 50  0000 R CNN
+F 1 "G5V1" H 22645 15055 50  0000 R CNN
+F 2 "Peavey-EVH5150:Relay_SPDT_Omron_G5V-1" H 22800 15100 50  0001 C CNN
+F 3 "" H 22800 15100 50  0001 C CNN
+	1    22800 15100
+	1    0    0    -1
+$EndComp
+$Comp
+L Peavey_5150-rescue:G5V1-Relays-Peavey_5150-rescue K6
+U 1 1 5FCD95C4
+P 23150 15100
+F 0 "K6" H 22995 15146 50  0000 R CNN
+F 1 "G5V1" H 22995 15055 50  0000 R CNN
+F 2 "Peavey-EVH5150:Relay_SPDT_Omron_G5V-1" H 23150 15100 50  0001 C CNN
+F 3 "" H 23150 15100 50  0001 C CNN
+	1    23150 15100
+	-1   0    0    -1
+$EndComp
+Wire Wire Line
+	22800 14800 22800 14700
+Connection ~ 22800 14700
+Wire Wire Line
+	22800 14700 22250 14700
+Wire Wire Line
+	22800 15400 22800 15500
+Connection ~ 22800 15500
+Wire Wire Line
+	22800 15500 23150 15500
+Text Notes 22300 15250 0    20   ~ 0
+12V 41.7mA
+Text Notes 23200 15250 0    20   ~ 0
+12V 12.5mA
+Text Notes 22850 15250 0    20   ~ 0
+12V 12.5mA
 $EndSCHEMATC

Commit message: Wattage and voltage corrections
Parts:
- C11: value 0.047uF 450V -> 0.047uF 400V
- C15: value .1uF 250V -> .1uF 50V
- C21, C23, C28, C29, C30, C33, C34, C38: symbol Device:CP1 -> Peavey_5150-rescue:CP1-Device
- C26: value 22uF 25V -> 22uF 50V; symbol Device:CP1 -> Peavey_5150-rescue:CP1-Device
- CR1, CR10, CR11, CR2, CR3, CR4, CR8, CR9: symbol Diode:1N4007 -> Peavey_5150-rescue:1N4007-Diode
- D1, D7, D8, D9: symbol Device:D -> Peavey_5150-rescue:D-Device
- D2: symbol Device:D_Schottky -> Peavey_5150-rescue:D_Schottky-Device
- D3, D5, D6: symbol Device:LED -> Peavey_5150-rescue:LED-Device
- J2: symbol Connector:Screw_Terminal_01x08 -> Peavey_5150-rescue:Screw_Terminal_01x08-Connector
- J4: symbol Connector_Generic:Conn_01x03 -> Peavey_5150-rescue:Conn_01x03-Connector_Generic
- JP1, JP2, JP3, JP4: symbol Device:Jumper_NC_Small -> Peavey_5150-rescue:Jumper_NC_Small-Device
- L1: symbol Device:L -> Peavey_5150-rescue:L-Device
- Q1: symbol Transistor_FET:IRF540N -> Peavey_5150-rescue:IRF540N-Transistor_FET
- Q2, Q3, Q4: symbol Transistor_BJT:BC847 -> Peavey_5150-rescue:BC847-Transistor_BJT
- R1, R3: value 100K -> 100K 1W; symbol Device:R_US -> Peavey_5150-rescue:R_US-Device
- R10, R28, R31, R34, R35, R37, R38, R42, R44, R45, R46, R47, R48, R49, R50, R51, R52, R53, R54, R55, R56, R57, R58, R61, R63, R65, R66, R67, R68, R8: symbol Device:R_US -> Peavey_5150-rescue:R_US-Device
- R101: value 100K -> 100K 1/2W; symbol Device:R_US -> Peavey_5150-rescue:R_US-Device
- R102, R93: value 2.2K 1/4W -> 2.2K 1/2W; symbol Device:R_US -> Peavey_5150-rescue:R_US-Device
- R103, R33: value 100K 1/4W -> 100K 1/2W; symbol Device:R_US -> Peavey_5150-rescue:R_US-Device
- R11: value 330K -> 330K 1/2W; symbol Device:R_US -> Peavey_5150-rescue:R_US-Device
- R12, R13, R17: value 1.82K 1/4W -> 1.82K 1/2W; symbol Device:R_US -> Peavey_5150-rescue:R_US-Device
- R14: value 3.3K 1/4W -> 3.3K 1/2W; symbol Device:R_US -> Peavey_5150-rescue:R_US-Device
- R15, R23: value 39K -> 39K 1/2W; symbol Device:R_US -> Peavey_5150-rescue:R_US-Device
- R16: value 100KW1 -> 100K 1W; symbol Device:R_US -> Peavey_5150-rescue:R_US-Device
- R160, R161, R25, R26, R41, R79: value 1M 1/4W -> 1M 1/2W; symbol Device:R_US -> Peavey_5150-rescue:R_US-Device
- R18, R94: value 47K -> 47K 1/2W; symbol Device:R_US -> Peavey_5150-rescue:R_US-Device
- R19, R6, R82, R89: value 470K -> 470K 1/2W; symbol Device:R_US -> Peavey_5150-rescue:R_US-Device
- R2, R4, R96: value 220K 1/4W -> 220K 1W; symbol Device:R_US -> Peavey_5150-rescue:R_US-Device
- R20, R7: value 220K -> 220K 1/2W; symbol Device:R_US -> Peavey_5150-rescue:R_US-Device
- R21, R32, R40, R87, R88, R9, R91: value 1M -> 1M 1/2W; symbol Device:R_US -> Peavey_5150-rescue:R_US-Device
- R22: value 68K 1/4W -> 68K 1/2W; symbol Device:R_US -> Peavey_5150-rescue:R_US-Device
- R24: value 33K -> 33K 1/2W; symbol Device:R_US -> Peavey_5150-rescue:R_US-Device
- R27: value 10K -> 10K 1/2W; symbol Device:R_US -> Peavey_5150-rescue:R_US-Device
- R29: value 470K 1/4W -> 470K 1/2W; symbol Device:R_US -> Peavey_5150-rescue:R_US-Device
- R30: value 22K 1/4W -> 22K 1/2W; symbol Device:R_US -> Peavey_5150-rescue:R_US-Device
- R36, R39: value 47R1W -> 47R 1W; symbol Device:R_US -> Peavey_5150-rescue:R_US-Device
- R43: value 2.2K -> 2.2K 1/2W; symbol Device:R_US -> Peavey_5150-rescue:R_US-Device
- R5: value 68K 1/4W -> 68K 1W; symbol Device:R_US -> Peavey_5150-rescue:R_US-Device
- R62, R64: value 220K 1W -> 220K 1W SMD; symbol Device:R_US -> Peavey_5150-rescue:R_US-Device
- R75: value 2.2M -> 2.2M 1/2W; symbol Device:R_US -> Peavey_5150-rescue:R_US-Device
- R80: value 1K 1/4W -> 1K 1/2W; symbol Device:R_US -> Peavey_5150-rescue:R_US-Device
- R81: value 2.2M 1/4W -> 2.2M 1/2W; symbol Device:R_US -> Peavey_5150-rescue:R_US-Device
- R85: value 220K 1/4W -> 220K 1/2W; symbol Device:R_US -> Peavey_5150-rescue:R_US-Device
- R86: value 100K 1/4W -> 100K 1W; symbol Device:R_US -> Peavey_5150-rescue:R_US-Device
- SW2, SW3, SW4: symbol Switch:SW_Push -> Peavey_5150-rescue:SW_Push-Switch
- U2: symbol Regulator_Linear:LT1129-3.3_SOT223 -> Peavey_5150-rescue:LT1129-3.3_SOT223-Regulator_Linear
- U3: symbol MCU_ST_STM8:STM8S003F3P -> Peavey_5150-rescue:STM8S003F3P-MCU_ST_STM8
- U4: symbol Relay_SolidState:TLP222A -> Peavey_5150-rescue:TLP222A-Relay_SolidState
- V1, V2, V3, V5: symbol Valve:ECC83 -> Peavey_5150-rescue:ECC83-Valve
- VR1, VR2, VR6, VR7: value 1M -> 1M LOG
Connections:
- net at C18.2, VR3.3, VR5.1: now also VR3.2
- no-connect marks 9 -> 8
