File: Peavey_5150.sch (KiCad schematic (older format))
At the start: 203 parts, among them J165 SEND, J166 RETURN, J2 Power, J3 OUTPUT, J37 INPUT FRONT, J39 INPUT REAR, J4 SWIM, J5 FOOTSWITCH, K1 G5V-2, K2 G5V1, K3 G5V-2, K4 G5V-2, K5 G5V1, K6 G5V1, Q1 IRF840, Q2 BC847, Q3 BC847, Q4 BC847, SW2 Clean, SW3 Bright, SW4 FX_loop, U1 MP4462, U2 AMS1117-3.3, U3 STM8S003F3P, U4 TLP222A

Commit message: move rescue lib
Parts:
- C1, C10, C11, C12, C13, C14, C15, C158, C16, C17, C18, C19, C2, C20, C22, C24, C25, C27, C3, C31, C32, C35, C36, C37, C39, C4, C40, C41, C42, C43, C45, C48, C49, C5, C51, C52, C53, C56, C57, C58, C59, C6, C63, C65, C7, C8, C9: symbol Peavey_5150-rescue:C_US-simple-Peavey_5150-rescue -> Peavey_5150:C_US-simple-Peavey_5150
- C21, C23, C26, C28, C29, C30, C33, C34, C38: symbol Peavey_5150-rescue:CP1-Device -> Peavey_5150:CP1-Device
- CR1, CR10, CR11, CR2, CR3, CR4, CR8, CR9: symbol Peavey_5150-rescue:1N4007-Diode -> Peavey_5150:1N4007-Diode
- D1, D7, D8, D9: symbol Peavey_5150-rescue:D-Device -> Peavey_5150:D-Device
- D2: symbol Peavey_5150-rescue:D_Schottky-Device -> Peavey_5150:D_Schottky-Device
- D3, D5, D6: symbol Peavey_5150-rescue:LED-Device -> Peavey_5150:LED-Device
- F1, F2: symbol Peavey_5150-rescue:Fuse-simple-Peavey_5150-rescue -> Peavey_5150:Fuse-simple-Peavey_5150
- J165, J166, J3, J37, J39, J5: symbol Peavey_5150-rescue:Jack_6.35-simple-Peavey_5150-rescue -> Peavey_5150:Jack_6.35-simple-Peavey_5150
- J2: symbol Peavey_5150-rescue:Screw_Terminal_01x08-Connector -> Peavey_5150:Screw_Terminal_01x08-Connector
- J4: symbol Peavey_5150-rescue:Conn_01x03-Connector_Generic -> Peavey_5150:Conn_01x03-Connector_Generic
- JP1, JP2, JP3, JP4: symbol Peavey_5150-rescue:Jumper_NC_Small-Device -> Peavey_5150:Jumper_NC_Small-Device
- K1, K3, K4: symbol Peavey_5150-rescue:G5V-2-Relays-Peavey_5150-rescue -> Peavey_5150:G5V-2-Relays-Peavey_5150
- K2, K5, K6: symbol Peavey_5150-rescue:G5V1-Relays-Peavey_5150-rescue -> Peavey_5150:G5V1-Relays-Peavey_5150
- L1: symbol Peavey_5150-rescue:L-Device -> Peavey_5150:L-Device
- Q1: symbol Peavey_5150-rescue:IRF540N-Transistor_FET -> Peavey_5150:IRF540N-Transistor_FET
- Q2, Q3, Q4: symbol Peavey_5150-rescue:BC847-Transistor_BJT -> Peavey_5150:BC847-Transistor_BJT
- R1, R10, R101, R102, R103, R11, R12, R13, R14, R15, R16, R160, R161, R17, R18, R19, R2, R20, R21, R22, R23, R24, R25, R26, R27, R28, R29, R3, R30, R31, R32, R33, R34, R35, R36, R37, R38, R39, R4, R40, R41, R42, R43, R44, R45, R46, R47, R48, R49, R5, R50, R51, R52, R53, R54, R55, R56, R57, R58, R6, R61, R62, R63, R64, R65, R66, R67, R68, R7, R75, R79, R8, R80, R81, R82, R85, R86, R87, R88, R89, R9, R91, R93, R94, R96: symbol Peavey_5150-rescue:R_US-Device -> Peavey_5150:R_US-Device
- SW2, SW3, SW4: symbol Peavey_5150-rescue:SW_Push-Switch -> Peavey_5150:SW_Push-Switch
- U1: symbol Peavey_5150-rescue:MP4462-simple-Peavey_5150-rescue -> Peavey_5150:MP4462-simple-Peavey_5150
- U2: symbol Peavey_5150-rescue:LT1129-3.3_SOT223-Regulator_Linear -> Peavey_5150:LT1129-3.3_SOT223-Regulator_Linear
- U3: symbol Peavey_5150-rescue:STM8S003F3P-MCU_ST_STM8 -> Peavey_5150:STM8S003F3P-MCU_ST_STM8
- U4: symbol Peavey_5150-rescue:TLP222A-Relay_SolidState -> Peavey_5150:TLP222A-Relay_SolidState
- V1, V2, V3, V5: symbol Peavey_5150-rescue:ECC83-Valve -> Peavey_5150:ECC83-Valve
- VR1, VR11, VR12, VR13, VR2, VR3, VR4, VR5, VR6, VR7: symbol Peavey_5150-rescue:R_POT_US_P-simple-Peavey_5150-rescue -> Peavey_5150:R_POT_US_P-simple-Peavey_5150
