File: Peavey_5150.sch (KiCad schematic (older format))
At the start: 203 parts, among them J165 SEND, J166 RETURN, J2 Power, J3 OUTPUT, J37 INPUT FRONT, J39 INPUT REAR, J4 SWIM, J5 FOOTSWITCH, K1 G5V-2, K2 G5V1, K3 G5V-2, K4 G5V-2, K5 G5V1, K6 G5V1, Q1 IRF840, Q2 BC847, Q3 BC847, Q4 BC847, SW2 Clean, SW3 Bright, SW4 FX_loop, U1 MP4462, U2 AMS1117-3.3, U3 STM8S003F3P, U4 TLP222A

Commit message: Common Lib
Parts:
- C1, C10, C11, C12, C13, C14, C15, C158, C16, C17, C18, C19, C2, C20, C22, C24, C25, C27, C3, C31, C32, C35, C36, C37, C39, C4, C40, C41, C42, C43, C45, C48, C49, C5, C51, C52, C53, C56, C57, C58, C59, C6, C63, C65, C7, C8, C9: symbol Peavey_5150:C_US-simple-Peavey_5150 -> KiCadCommon:C_US-simple-KiCadCommon
- C21, C23, C26, C28, C29, C30, C33, C34, C38: symbol Peavey_5150:CP1-Device -> KiCadCommon:CP1-Device
- CR1, CR10, CR11, CR2, CR3, CR4, CR8, CR9: symbol Peavey_5150:1N4007-Diode -> KiCadCommon:1N4007-Diode
- D1, D7, D8, D9: symbol Peavey_5150:D-Device -> KiCadCommon:D-Device
- D2: symbol Peavey_5150:D_Schottky-Device -> KiCadCommon:D_Schottky-Device
- D3, D5, D6: symbol Peavey_5150:LED-Device -> KiCadCommon:LED-Device
- F1, F2: symbol Peavey_5150:Fuse-simple-Peavey_5150 -> KiCadCommon:Fuse-simple-KiCadCommon
- J165, J166, J3, J37, J39, J5: symbol Peavey_5150:Jack_6.35-simple-Peavey_5150 -> KiCadCommon:Jack_6.35-simple-KiCadCommon
- J2: symbol Peavey_5150:Screw_Terminal_01x08-Connector -> KiCadCommon:Screw_Terminal_01x08-Connector
- J4: symbol Peavey_5150:Conn_01x03-Connector_Generic -> KiCadCommon:Conn_01x03-Connector_Generic
- JP1, JP2, JP3, JP4: symbol Peavey_5150:Jumper_NC_Small-Device -> KiCadCommon:Jumper_NC_Small-Device
- K1, K3, K4: symbol Peavey_5150:G5V-2-Relays-Peavey_5150 -> KiCadCommon:G5V-2-Relays-KiCadCommon
- K2, K5, K6: symbol Peavey_5150:G5V1-Relays-Peavey_5150 -> KiCadCommon:G5V1-Relays-KiCadCommon
- L1: symbol Peavey_5150:L-Device -> KiCadCommon:L-Device
- Q1: symbol Peavey_5150:IRF540N-Transistor_FET -> KiCadCommon:IRF540N-Transistor_FET
- Q2, Q3, Q4: symbol Peavey_5150:BC847-Transistor_BJT -> KiCadCommon:BC847-Transistor_BJT
- R1, R10, R101, R102, R103, R11, R12, R13, R14, R15, R16, R160, R161, R17, R18, R19, R2, R20, R21, R22, R23, R24, R25, R26, R27, R28, R29, R3, R30, R31, R32, R33, R34, R35, R36, R37, R38, R39, R4, R40, R41, R42, R43, R44, R45, R46, R47, R48, R49, R5, R50, R51, R52, R53, R54, R55, R56, R57, R58, R6, R61, R62, R63, R64, R65, R66, R67, R68, R7, R75, R79, R8, R80, R81, R82, R85, R86, R87, R88, R89, R9, R91, R93, R94, R96: symbol Peavey_5150:R_US-Device -> KiCadCommon:R_US-Device
- SW2, SW3, SW4: symbol Peavey_5150:SW_Push-Switch -> KiCadCommon:SW_Push-Switch
- U1: symbol Peavey_5150:MP4462-simple-Peavey_5150 -> KiCadCommon:MP4462-simple-KiCadCommon
- U2: symbol Peavey_5150:LT1129-3.3_SOT223-Regulator_Linear -> KiCadCommon:LT1129-3.3_SOT223-Regulator_Linear
- U3: symbol Peavey_5150:STM8S003F3P-MCU_ST_STM8 -> KiCadCommon:STM8S003F3P-MCU_ST_STM8
- U4: symbol Peavey_5150:TLP222A-Relay_SolidState -> KiCadCommon:TLP222A-Relay_SolidState
- V1, V2, V3, V5: symbol Peavey_5150:ECC83-Valve -> KiCadCommon:ECC83-Valve
- VR1, VR11, VR12, VR13, VR2, VR3, VR4, VR5, VR6, VR7: symbol Peavey_5150:R_POT_US_P-simple-Peavey_5150 -> KiCadCommon:R_POT_US_P-simple-KiCadCommon

Commit message: Prettify
Parts:
- C1, C2, C6: footprint Peavey-EVH5150:C_UNIVERSAL -> KiCadCommon:KiCadCommon_C_Horizontal_MP
- C3, C4, C5: footprint Peavey-EVH5150:CP_UNIVERSAL -> KiCadCommon:KiCadCommon_CP_Vertical_MP
Connections:
- wire segments 729 -> 731
Other:
- note added: "(install jumpers for 6N2P tubes)"
- note added: "Ground Wiring"
- note added: "High Voltage PSU"
- note added: "Low Voltage PSU"
- note added: "Operation"
- note added: "Power Connector"
- note added: "Relay wiring"
- note added: "Tube heater"
- note removed: "Relay power"
- note removed: "Tube heat (put jumper for 6N2P)"

Commit message: Clenup / footprint assignment
Parts:
- C49, C56, C57, C58: footprint Peavey-EVH5150:C_UNIVERSAL -> KiCadCommon:KiCadCommon_C_Horizontal_MP
- J165, J166, J3, J37, J39, J5: footprint Peavey-EVH5150:Jack_6.35 -> KiCadCommon:KiCadCommon_Jack_Horizontal_6.35mm
- J2: footprint Peavey-EVH5150:X977T08 -> KiCadCommon:KiCadCommon_TerminalBlock_X977T08
- K1, K3, K4: footprint Peavey-EVH5150:Relay_DPDT_Omron_G5V-2 -> KiCadCommon:KiCadCommon_Relay_DPDT_Omron_G5V-2
- K2, K5, K6: footprint Peavey-EVH5150:Relay_SPDT_Omron_G5V-1 -> KiCadCommon:KiCadCommon_Relay_SPDT_Omron_G5V-1
- R12, R13, R14, R15: footprint (none) -> KiCadCommon:KiCadCommon_R_Vertical_L9.0mm_D3.2mm_P2.54mm
- V1, V2, V3, V5: footprint Peavey-EVH5150:GZC9-A -> KiCadCommon:KiCadCommon_Tube_Socket_MP
- VR1, VR12, VR13, VR2, VR3, VR4, VR5, VR6, VR7: footprint (none) -> KiCadCommon:KiCadCommon_Potentiometer_Alpha_Single_Horizontal

Commit message: Up
Parts:
- C10, C13, C14, C51: footprint (none) -> KiCadCommon:KiCadCommon_C_Rect_L7.2mm_W5.5mm_P5.00mm_Wima_Fat
- C11, C52, C53, C65: footprint (none) -> KiCadCommon:KiCadCommon_C_Horizontal_MP
- C158: footprint (none) -> KiCadCommon:KiCadCommon_CP_Vertical_MP
- C17, C18, C37: footprint (none) -> KiCadCommon:KiCadCommon_C_Rect_L7.2mm_W3.0mm_P5.00mm_Wima_Slim
- C19, C27, C48, C59, C63: footprint (none) -> KiCadCommon:KiCadCommon_C_Rect_L7.2mm_W4.5mm_P5.00mm_Wima_Small
- R1, R16, R2, R3, R4, R5, R9: footprint (none) -> KiCadCommon:KiCadCommon_R_Axial_1W
- R11, R17, R18, R19, R20, R21, R22, R23, R24, R25, R26, R27, R6, R7: footprint (none) -> KiCadCommon:KiCadCommon_R_Axial_0.5W
Changed lines of the file:
@@
 F 0 "R24" H 20168 5204 50  0000 L CNN
 F 1 "33K 1/2W" H 20168 5295 50  0000 L CNN
-F 2 "" V 20140 5240 50  0001 C CNN
+F 2 "KiCadCommon:KiCadCommon_R_Axial_0.5W" V 20140 5240 50  0001 C CNN
 F 3 "~" H 20100 5250 50  0001 C CNN
 	1    20100 5250
@@
 F 0 "C59" H 20400 5150 50  0000 L CNN
 F 1 "0.01uF 50v" H 20400 4950 50  0000 L CNN
-F 2 "" H 20350 5050 50  0001 C CNN
+F 2 "KiCadCommon:KiCadCommon_C_Rect_L7.2mm_W4.5mm_P5.00mm_Wima_Small" H 20350 5050 50  0001 C CNN
 F 3 "" H 20350 5050 50  0001 C CNN
 	1    20350 5050
@@
 F 0 "C37" H 21450 6300 50  0000 L CNN
 F 1 "0.022uF 50v" H 21450 6100 50  0000 L CNN
-F 2 "" H 21400 6200 50  0001 C CNN
+F 2 "KiCadCommon:KiCadCommon_C_Rect_L7.2mm_W3.0mm_P5.00mm_Wima_Slim" H 21400 6200 50  0001 C CNN
 F 3 "" H 21400 6200 50  0001 C CNN
 	1    21400 6200
@@
 F 0 "C14" V 22200 4750 50  0000 L CNN
 F 1 "470pF 50v" V 21900 4650 50  0000 L CNN
-F 2 "" H 22050 4800 50  0001 C CNN
+F 2 "KiCadCommon:KiCadCommon_C_Rect_L7.2mm_W5.5mm_P5.00mm_Wima_Fat" H 22050 4800 50  0001 C CNN
 F 3 "" H 22050 4800 50  0001 C CNN
 	1    22050 4800
@@
 F 0 "C18" V 22050 5650 50  0000 L CNN
 F 1 "0.022uF 50v" V 21750 5550 50  0000 L CNN
-F 2 "" H 21900 5700 50  0001 C CNN
+F 2 "KiCadCommon:KiCadCommon_C_Rect_L7.2mm_W3.0mm_P5.00mm_Wima_Slim" H 21900 5700 50  0001 C CNN
 F 3 "" H 21900 5700 50  0001 C CNN
 	1    21900 5700
@@
 F 0 "R16" H 26232 6104 50  0000 R CNN
 F 1 "100K 1W" H 26232 6195 50  0000 R CNN
-F 2 "" V 26340 6140 50  0001 C CNN
+F 2 "KiCadCommon:KiCadCommon_R_Axial_1W" V 26340 6140 50  0001 C CNN
 F 3 "~" H 26300 6150 50  0001 C CNN
 	1    26300 6150
@@
 F 0 "C53" V 26850 5200 50  0000 L CNN
 F 1 "0.33uF 400v" V 26550 5150 50  0000 L CNN
-F 2 "" H 26700 5300 50  0001 C CNN
+F 2 "KiCadCommon:KiCadCommon_C_Horizontal_MP" H 26700 5300 50  0001 C CNN
 F 3 "" H 26700 5300 50  0001 C CNN
 	1    26700 5300
@@
 F 0 "C65" V 27550 5200 50  0000 L CNN
 F 1 "0.33uF 400v" V 27250 5150 50  0000 L CNN
-F 2 "" H 27400 5300 50  0001 C CNN
+F 2 "KiCadCommon:KiCadCommon_C_Horizontal_MP" H 27400 5300 50  0001 C CNN
 F 3 "" H 27400 5300 50  0001 C CNN
 	1    27400 5300
@@
 F 0 "C11" V 27550 7900 50  0000 L CNN
 F 1 "0.047uF 400V" V 27250 7850 50  0000 L CNN
-F 2 "" H 27400 8000 50  0001 C CNN
+F 2 "KiCadCommon:KiCadCommon_C_Horizontal_MP" H 27400 8000 50  0001 C CNN
 F 3 "" H 27400 8000 50  0001 C CNN
 	1    27400 8000
@@
 F 0 "R26" H 26950 8350 50  0000 L CNN
 F 1 "1M 1/2W" H 26950 8450 50  0000 L CNN
-F 2 "" V 26940 8390 50  0001 C CNN
+F 2 "KiCadCommon:KiCadCommon_R_Axial_0.5W" V 26940 8390 50  0001 C CNN
 F 3 "~" H 26900 8400 50  0001 C CNN
 	1    26900 8400
@@
 F 0 "R5" H 26250 7200 50  0000 L CNN
 F 1 "68K 1W" H 26250 7300 50  0000 L CNN
-F 2 "" V 26240 7240 50  0001 C CNN
+F 2 "KiCadCommon:KiCadCommon_R_Axial_1W" V 26240 7240 50  0001 C CNN
 F 3 "~" H 26200 7250 50  0001 C CNN
 	1    26200 7250
@@
 F 0 "C158" H 26050 8850 50  0000 R CNN
 F 1 "0.0047uF 50v" H 26050 8650 50  0000 R CNN
-F 2 "" H 26100 8750 50  0001 C CNN
+F 2 "KiCadCommon:KiCadCommon_CP_Vertical_MP" H 26100 8750 50  0001 C CNN
 F 3 "" H 26100 8750 50  0001 C CNN
 	1    26100 8750
@@
 F 0 "C19" H 6950 5950 50  0000 L CNN
 F 1 ".001uf 50V" H 6950 5750 50  0000 L CNN
-F 2 "" H 6900 5850 50  0001 C CNN
+F 2 "KiCadCommon:KiCadCommon_C_Rect_L7.2mm_W4.5mm_P5.00mm_Wima_Small" H 6900 5850 50  0001 C CNN
 F 3 "" H 6900 5850 50  0001 C CNN
 	1    6900 5850
@@
 F 0 "C17" H 6950 4850 50  0000 L CNN
 F 1 ".0022uF 50v" H 6950 4650 50  0000 L CNN
-F 2 "" H 6900 4750 50  0001 C CNN
+F 2 "KiCadCommon:KiCadCommon_C_Rect_L7.2mm_W3.0mm_P5.00mm_Wima_Slim" H 6900 4750 50  0001 C CNN
 F 3 "" H 6900 4750 50  0001 C CNN
 	1    6900 4750
@@
 F 0 "C27" V 8650 5250 50  0000 C CNN
 F 1 "180pF 50V" V 8350 5250 50  0000 C CNN
-F 2 "" H 8500 5250 50  0001 C CNN
+F 2 "KiCadCommon:KiCadCommon_C_Rect_L7.2mm_W4.5mm_P5.00mm_Wima_Small" H 8500 5250 50  0001 C CNN
 F 3 "" H 8500 5250 50  0001 C CNN
 	1    8500 5250
@@
 F 0 "C13" V 8850 3150 50  0000 C CNN
 F 1 "470pF 50V" V 8550 3150 50  0000 C CNN
-F 2 "" H 8700 3150 50  0001 C CNN
+F 2 "KiCadCommon:KiCadCommon_C_Rect_L7.2mm_W5.5mm_P5.00mm_Wima_Fat" H 8700 3150 50  0001 C CNN
 F 3 "" H 8700 3150 50  0001 C CNN
 	1    8700 3150
@@
 F 0 "C10" H 9050 4050 50  0000 R CNN
 F 1 "470pF 50V" H 9050 3900 50  0000 R CNN
-F 2 "" H 9150 4000 50  0001 C CNN
+F 2 "KiCadCommon:KiCadCommon_C_Rect_L7.2mm_W5.5mm_P5.00mm_Wima_Fat" H 9150 4000 50  0001 C CNN
 F 3 "" H 9150 4000 50  0001 C CNN
 	1    9150 4000
@@
 F 0 "C63" V 7050 4150 50  0000 C CNN
 F 1 ".1uF 50V" V 6750 4150 50  0000 C CNN
-F 2 "" H 6900 4150 50  0001 C CNN
+F 2 "KiCadCommon:KiCadCommon_C_Rect_L7.2mm_W4.5mm_P5.00mm_Wima_Small" H 6900 4150 50  0001 C CNN
 F 3 "" H 6900 4150 50  0001 C CNN
 	1    6900 4150
@@
 F 0 "R23" V 7200 4150 50  0000 C CNN
 F 1 "39K 1/2W" V 7400 4150 50  0000 C CNN
-F 2 "" V 7340 4140 50  0001 C CNN
+F 2 "KiCadCommon:KiCadCommon_R_Axial_0.5W" V 7340 4140 50  0001 C CNN
 F 3 "~" H 7300 4150 50  0001 C CNN
 	1    7300 4150
@@
 F 0 "R21" H 8200 3950 50  0000 R CNN
 F 1 "1M 1/2W" H 8200 4050 50  0000 R CNN
-F 2 "" V 8290 3990 50  0001 C CNN
+F 2 "KiCadCommon:KiCadCommon_R_Axial_0.5W" V 8290 3990 50  0001 C CNN
 F 3 "~" H 8250 4000 50  0001 C CNN
 	1    8250 4000
@@
 F 0 "C51" V 8150 3350 50  0000 C CNN
 F 1 "270pF 50V" V 7850 3350 50  0000 C CNN
-F 2 "" H 8000 3350 50  0001 C CNN
+F 2 "KiCadCommon:KiCadCommon_C_Rect_L7.2mm_W5.5mm_P5.00mm_Wima_Fat" H 8000 3350 50  0001 C CNN
 F 3 "" H 8000 3350 50  0001 C CNN
 	1    8000 3350
@@
 F 0 "R19" V 7900 3750 50  0000 C CNN
 F 1 "470K 1/2W" V 8100 3750 50  0000 C CNN
-F 2 "" V 8040 3740 50  0001 C CNN
+F 2 "KiCadCommon:KiCadCommon_R_Axial_0.5W" V 8040 3740 50  0001 C CNN
 F 3 "~" H 8000 3750 50  0001 C CNN
 	1    8000 3750
@@
 F 0 "R2" H 5200 3250 50  0000 R CNN
 F 1 "220K 1W" H 5200 3350 50  0000 R CNN
-F 2 "" V 5290 3290 50  0001 C CNN
+F 2 "KiCadCommon:KiCadCommon_R_Axial_1W" V 5290 3290 50  0001 C CNN
 F 3 "~" H 5250 3300 50  0001 C CNN
 	1    5250 3300
@@
 F 0 "R22" H 4150 4350 50  0000 R CNN
 F 1 "68K 1/2W" H 4150 4450 50  0000 R CNN
-F 2 "" V 4240 4390 50  0001 C CNN
+F 2 "KiCadCommon:KiCadCommon_R_Axial_0.5W" V 4240 4390 50  0001 C CNN
 F 3 "~" H 4200 4400 50  0001 C CNN
 	1    4200 4400
@@
 F 0 "R25" V 3750 4650 50  0000 C CNN
 F 1 "1M 1/2W" V 3950 4650 50  0000 C CNN
-F 2 "" V 3890 4640 50  0001 C CNN
+F 2 "KiCadCommon:KiCadCommon_R_Axial_0.5W" V 3890 4640 50  0001 C CNN
 F 3 "~" H 3850 4650 50  0001 C CNN
 	1    3850 4650
@@
 F 0 "R3" H 10450 3750 50  0000 R CNN
 F 1 "100K 1W" H 10450 3850 50  0000 R CNN
-F 2 "" V 10540 3790 50  0001 C CNN
+F 2 "KiCadCommon:KiCadCommon_R_Axial_1W" V 10540 3790 50  0001 C CNN
 F 3 "~" H 10500 3800 50  0001 C CNN
 	1    10500 3800
@@
 F 0 "R17" H 10350 5350 50  0000 R CNN
 F 1 "1.82K 1/2W" H 10350 5450 50  0000 R CNN
-F 2 "" V 10440 5390 50  0001 C CNN
+F 2 "KiCadCommon:KiCadCommon_R_Axial_0.5W" V 10440 5390 50  0001 C CNN
 F 3 "~" H 10400 5400 50  0001 C CNN
 	1    10400 5400
@@
 F 0 "R6" H 11350 4350 50  0000 R CNN
 F 1 "470K 1/2W" H 11350 4450 50  0000 R CNN
-F 2 "" V 11440 4390 50  0001 C CNN
+F 2 "KiCadCommon:KiCadCommon_R_Axial_0.5W" V 11440 4390 50  0001 C CNN
 F 3 "~" H 11400 4400 50  0001 C CNN
 	1    11400 4400
@@
 F 0 "R9" H 11468 4854 50  0000 L CNN
 F 1 "1M 1/2W" H 11468 4945 50  0000 L CNN
-F 2 "" V 11440 4890 50  0001 C CNN
+F 2 "KiCadCommon:KiCadCommon_R_Axial_1W" V 11440 4890 50  0001 C CNN
 F 3 "~" H 11400 4900 50  0001 C CNN
 	1    11400 4900
@@
 F 0 "R20" H 11650 5800 50  0000 R CNN
 F 1 "220K 1/2W" H 11650 5900 50  0000 R CNN
-F 2 "" V 11740 5840 50  0001 C CNN
+F 2 "KiCadCommon:KiCadCommon_R_Axial_0.5W" V 11740 5840 50  0001 C CNN
 F 3 "~" H 11700 5850 50  0001 C CNN
 	1    11700 5850
@@
 F 0 "R18" H 11000 6750 50  0000 R CNN
 F 1 "47K 1/2W" H 11000 6850 50  0000 R CNN
-F 2 "" V 11090 6790 50  0001 C CNN
+F 2 "KiCadCommon:KiCadCommon_R_Axial_0.5W" V 11090 6790 50  0001 C CNN
 F 3 "~" H 11050 6800 50  0001 C CNN
 	1    11050 6800
@@
 F 0 "R1" H 12150 3750 50  0000 R CNN
 F 1 "100K 1W" H 12150 3850 50  0000 R CNN
-F 2 "" V 12240 3790 50  0001 C CNN
+F 2 "KiCadCommon:KiCadCommon_R_Axial_1W" V 12240 3790 50  0001 C CNN
 F 3 "~" H 12200 3800 50  0001 C CNN
 	1    12200 3800
@@
 F 0 "R11" H 13300 4850 50  0000 R CNN
 F 1 "330K 1/2W" H 13300 4950 50  0000 R CNN
-F 2 "" V 13390 4890 50  0001 C CNN
+F 2 "KiCadCommon:KiCadCommon_R_Axial_0.5W" V 13390 4890 50  0001 C CNN
 F 3 "~" H 13350 4900 50  0001 C CNN
 	1    13350 4900
@@
 F 0 "C48" H 13050 4950 50  0000 R CNN
 F 1 ".001uf 50V" H 13050 4800 50  0000 R CNN
-F 2 "" H 13150 4900 50  0001 C CNN
+F 2 "KiCadCommon:KiCadCommon_C_Rect_L7.2mm_W4.5mm_P5.00mm_Wima_Small" H 13150 4900 50  0001 C CNN
 F 3 "" H 13150 4900 50  0001 C CNN
 	1    13150 4900
@@
 F 0 "R7" V 13650 4650 50  0000 C CNN
 F 1 "220K 1/2W" V 13850 4650 50  0000 C CNN
-F 2 "" V 13790 4640 50  0001 C CNN
+F 2 "KiCadCommon:KiCadCommon_R_Axial_0.5W" V 13790 4640 50  0001 C CNN
 F 3 "~" H 13750 4650 50  0001 C CNN
 	1    13750 4650
@@
 F 0 "R4" H 14250 3750 50  0000 R CNN
 F 1 "220K 1W" H 14250 3850 50  0000 R CNN
-F 2 "" V 14340 3790 50  0001 C CNN
+F 2 "KiCadCommon:KiCadCommon_R_Axial_1W" V 14340 3790 50  0001 C CNN
 F 3 "~" H 14300 3800 50  0001 C CNN
 	1    14300 3800
@@
 F 0 "C52" V 25450 4750 50  0000 L CNN
 F 1 ".022uF 400V" V 25150 4500 50  0000 L CNN
-F 2 "" H 25300 4800 50  0001 C CNN
+F 2 "KiCadCommon:KiCadCommon_C_Horizontal_MP" H 25300 4800 50  0001 C CNN
 F 3 "" H 25300 4800 50  0001 C CNN
 	1    25300 4800
@@
 F 0 "R27" H 21468 5404 50  0000 L CNN
 F 1 "10K 1/2W" H 21468 5495 50  0000 L CNN
-F 2 "" V 21440 5440 50  0001 C CNN
+F 2 "KiCadCommon:KiCadCommon_R_Axial_0.5W" V 21440 5440 50  0001 C CNN
 F 3 "~" H 21400 5450 50  0001 C CNN
 	1    21400 5450

Commit message: Annotation
Parts:
- renumbered C20 to C1, C17 to C10, C32 to C100, C7 to C101, C8 to C102, C12 to C103, C16 to C104, C34 to C105, C38 to C106, C23 to C107, C25 to C108, C29 to C109, C19 to C11, C30 to C110, C33 to C111, C4 to C12, C26 to C13, C2 to C14, C1 to C15, C48 to C16, C5 to C17, C57 to C18, C56 to C19, C15 to C2, C58 to C20, C9 to C200, C21 to C201, C24 to C202, C22 to C203, C31 to C204, C28 to C205, C35 to C206, C36 to C207, C59 to C21, C14 to C22, C18 to C23, C37 to C24, C52 to C25, C53 to C26, C65 to C27, C11 to C28, C158 to C29, C49 to C30, C39 to C300, C40 to C301, C41 to C302, C42 to C303, C43 to C304, C45 to C305, C6 to C4, C13 to C5, C51 to C6, C10 to C7, C63 to C8, C27 to C9, CR8 to CR100, CR9 to CR101, CR11 to CR102, CR10 to CR103, CR1 to CR200, CR3 to CR201, CR2 to CR202, CR4 to CR203, D1 to D104, D2 to D200, D7 to D300, D8 to D301, D9 to D302, D6 to D303, D3 to D304, D5 to D305, F1 to F100, F2 to F200, J37 to J1, J2 to J10, J39 to J2, J165 to J3, J4 to J300, J166 to J4, J3 to J5, J5 to J6, JP1 to JP100, JP2 to JP101, JP3 to JP102, JP4 to JP103, K4 to K1, K5 to K2, K2 to K3, K1 to K4, K6 to K5, K3 to K6, L1 to L200, Q1 to Q100, Q2 to Q300, Q3 to Q301, Q4 to Q302, R30 to R1, R23 to R10, R62 to R100, R64 to R101, R63 to R102, R65 to R103, R66 to R104, R67 to R105, R31 to R106, R35 to R107, R38 to R108, R29 to R11, R41 to R12, R40 to R13, R82 to R14, R17 to R15, R18 to R16, R3 to R17, R6 to R18, R9 to R19, R25 to R2, R8 to R200, R10 to R201, R37 to R202, R28 to R203, R34 to R204, R15 to R21, R1 to R22, R11 to R23, R7 to R24, R13 to R25, R4 to R26, R32 to R27, R101 to R28, R102 to R29, R22 to R3, R96 to R30, R42 to R300, R68 to R301, R46 to R303, R49 to R304, R52 to R305, R44 to R306, R45 to R307, R47 to R308, R48 to R309, R87 to R31, R50 to R310, R51 to R311, R54 to R312, R55 to R313, R57 to R314, R61 to R315, R58 to R316, R56 to R317, R53 to R318, R91 to R32, R88 to R33, R93 to R34, R86 to R35, R89 to R36, R24 to R37, R94 to R38, R27 to R39, R12 to R4, R81 to R40, R79 to R41, R80 to R42, R16 to R43, R103 to R44, R33 to R45, R160 to R46, R161 to R47, R85 to R48, R26 to R49, R2 to R5, R14 to R50, R5 to R51, R36 to R52, R39 to R53, R43 to R6, R19 to R7, R21 to R8, R75 to R9, SW2 to SW300, SW3 to SW301, SW4 to SW302, U4 to U1, U1 to U200, U2 to U201, U3 to U300, V5 to V3, V5 to V4, V3 to V4, VR11 to VR200, VR12 to VR3, VR5 to VR4, VR3 to VR5, VR4 to VR6, VR6 to VR7, VR7 to VR8, VR13 to VR9
Connections:
- wire segments 731 -> 730
