File: Peavey_5150.sch (KiCad schematic (older format))
At the start: 203 parts, among them J1 INPUT FRONT, J10 Power, J2 INPUT REAR, J3 SEND, J300 SWIM, J4 RETURN, J5 OUTPUT, J6 FOOTSWITCH, K1 G5V-2, K2 G5V1, K3 G5V1, K4 G5V-2, K5 G5V1, K6 G5V-2, Q100 IRF840, Q300 BC847, Q301 BC847, Q302 BC847, SW300 Clean, SW301 Bright, SW302 FX_loop, U1 TLP222A, U200 MP4462, U201 AMS1117-3.3, U300 STM8S003F3P

Commit message: Some footprints assigned
Parts:
- C1, C2: footprint (none) -> KiCadCommon:KiCadCommon_C_Rect_L7.2mm_W4.5mm_P5.00mm_Wima_Small
- R1, R11, R12, R13, R14, R27, R28, R31, R32, R33, R34, R36, R38, R40, R41, R42, R44, R45, R46, R47, R48, R9: footprint (none) -> KiCadCommon:KiCadCommon_R_Axial_0.5W
- R15, R16: footprint KiCadCommon:KiCadCommon_R_Axial_0.5W -> KiCadCommon:KiCadCommon_R_Vertical_L9.0mm_D3.2mm_P2.54mm
- R29, R6: footprint (none) -> KiCadCommon:KiCadCommon_R_Vertical_L9.0mm_D3.2mm_P2.54mm
- R30, R35, R52, R53: footprint (none) -> KiCadCommon:KiCadCommon_R_Axial_1W
Changed lines of the file:
@@
 F 0 "R38" H 20300 5300 50  0000 R CNN
 F 1 "47K 1/2W" H 20300 5400 50  0000 R CNN
-F 2 "" V 20390 5340 50  0001 C CNN
+F 2 "KiCadCommon:KiCadCommon_R_Axial_0.5W" V 20390 5340 50  0001 C CNN
 F 3 "~" H 20350 5350 50  0001 C CNN
 	1    20350 5350
@@
 F 0 "R41" H 25900 5100 50  0000 L CNN
 F 1 "1M 1/2W" H 25900 5200 50  0000 L CNN
-F 2 "" V 25890 5140 50  0001 C CNN
+F 2 "KiCadCommon:KiCadCommon_R_Axial_0.5W" V 25890 5140 50  0001 C CNN
 F 3 "~" H 25850 5150 50  0001 C CNN
 	1    25850 5150
@@
 F 0 "R42" H 26350 5600 50  0000 L CNN
 F 1 "1K 1/2W" H 26350 5700 50  0000 L CNN
-F 2 "" V 26340 5640 50  0001 C CNN
+F 2 "KiCadCommon:KiCadCommon_R_Axial_0.5W" V 26340 5640 50  0001 C CNN
 F 3 "~" H 26300 5650 50  0001 C CNN
 	1    26300 5650
@@
 F 0 "R40" H 25050 5250 50  0000 L CNN
 F 1 "2.2M 1/2W" H 25050 5350 50  0000 L CNN
-F 2 "" V 25040 5290 50  0001 C CNN
+F 2 "KiCadCommon:KiCadCommon_R_Axial_0.5W" V 25040 5290 50  0001 C CNN
 F 3 "~" H 25000 5300 50  0001 C CNN
 	1    25000 5300
@@
 F 0 "R44" H 27050 5600 50  0000 L CNN
 F 1 "100K 1/2W" H 27050 5700 50  0000 L CNN
-F 2 "" V 27040 5640 50  0001 C CNN
+F 2 "KiCadCommon:KiCadCommon_R_Axial_0.5W" V 27040 5640 50  0001 C CNN
 F 3 "~" H 27000 5650 50  0001 C CNN
 	1    27000 5650
@@
 F 0 "R45" H 27700 5600 50  0000 L CNN
 F 1 "100K 1/2W" H 27700 5700 50  0000 L CNN
-F 2 "" V 27690 5640 50  0001 C CNN
+F 2 "KiCadCommon:KiCadCommon_R_Axial_0.5W" V 27690 5640 50  0001 C CNN
 F 3 "~" H 27650 5650 50  0001 C CNN
 	1    27650 5650
@@
 F 0 "R46" H 28900 5400 50  0000 L CNN
 F 1 "1M 1/2W" H 28900 5500 50  0000 L CNN
-F 2 "" V 28890 5440 50  0001 C CNN
+F 2 "KiCadCommon:KiCadCommon_R_Axial_0.5W" V 28890 5440 50  0001 C CNN
 F 3 "~" H 28850 5450 50  0001 C CNN
 	1    28850 5450
@@
 F 0 "R47" H 28900 6300 50  0000 L CNN
 F 1 "1M 1/2W" H 28900 6400 50  0000 L CNN
-F 2 "" V 28890 6340 50  0001 C CNN
+F 2 "KiCadCommon:KiCadCommon_R_Axial_0.5W" V 28890 6340 50  0001 C CNN
 F 3 "~" H 28850 6350 50  0001 C CNN
 	1    28850 6350
@@
 F 0 "R48" H 27700 8350 50  0000 L CNN
 F 1 "220K 1/2W" H 27700 8450 50  0000 L CNN
-F 2 "" V 27690 8390 50  0001 C CNN
+F 2 "KiCadCommon:KiCadCommon_R_Axial_0.5W" V 27690 8390 50  0001 C CNN
 F 3 "~" H 27650 8400 50  0001 C CNN
 	1    27650 8400
@@
 F 0 "R53" V 4350 13600 50  0000 C CNN
 F 1 "47R 1W" V 4550 13600 50  0000 C CNN
-F 2 "" V 4490 13590 50  0001 C CNN
+F 2 "KiCadCommon:KiCadCommon_R_Axial_1W" V 4490 13590 50  0001 C CNN
 F 3 "~" H 4450 13600 50  0001 C CNN
 	1    4450 13600
@@
 F 0 "R52" V 3850 13600 50  0000 C CNN
 F 1 "47R 1W" V 4050 13600 50  0000 C CNN
-F 2 "" V 3990 13590 50  0001 C CNN
+F 2 "KiCadCommon:KiCadCommon_R_Axial_1W" V 3990 13590 50  0001 C CNN
 F 3 "~" H 3950 13600 50  0001 C CNN
 	1    3950 13600
@@
 F 0 "R12" H 5450 6050 50  0000 R CNN
 F 1 "1M 1/2W" H 5450 6150 50  0000 R CNN
-F 2 "" V 5540 6090 50  0001 C CNN
+F 2 "KiCadCommon:KiCadCommon_R_Axial_0.5W" V 5540 6090 50  0001 C CNN
 F 3 "~" H 5500 6100 50  0001 C CNN
 	1    5500 6100
@@
 F 0 "R13" H 7450 5800 50  0000 R CNN
 F 1 "1M 1/2W" H 7450 5900 50  0000 R CNN
-F 2 "" V 7540 5840 50  0001 C CNN
+F 2 "KiCadCommon:KiCadCommon_R_Axial_0.5W" V 7540 5840 50  0001 C CNN
 F 3 "~" H 7500 5850 50  0001 C CNN
 	1    7500 5850
@@
 F 0 "R11" H 6100 4700 50  0000 R CNN
 F 1 "470K 1/2W" H 6100 4800 50  0000 R CNN
-F 2 "" V 6190 4740 50  0001 C CNN
+F 2 "KiCadCommon:KiCadCommon_R_Axial_0.5W" V 6190 4740 50  0001 C CNN
 F 3 "~" H 6150 4750 50  0001 C CNN
 	1    6150 4750
@@
 F 0 "R9" V 8400 4250 50  0000 C CNN
 F 1 "2.2M 1/2W" V 8600 4250 50  0000 C CNN
-F 2 "" V 8540 4240 50  0001 C CNN
+F 2 "KiCadCommon:KiCadCommon_R_Axial_0.5W" V 8540 4240 50  0001 C CNN
 F 3 "~" H 8500 4250 50  0001 C CNN
 	1    8500 4250
@@
 F 0 "R6" V 8600 3550 50  0000 C CNN
 F 1 "2.2K 1/2W" V 8800 3550 50  0000 C CNN
-F 2 "" V 8740 3540 50  0001 C CNN
+F 2 "KiCadCommon:KiCadCommon_R_Vertical_L9.0mm_D3.2mm_P2.54mm" V 8740 3540 50  0001 C CNN
 F 3 "~" H 8700 3550 50  0001 C CNN
 	1    8700 3550
@@
 F 0 "C1" H 4100 6500 50  0000 R CNN
 F 1 "39pF 50V" H 4100 6400 50  0000 R CNN
-F 2 "" H 4200 6500 50  0001 C CNN
+F 2 "KiCadCommon:KiCadCommon_C_Rect_L7.2mm_W4.5mm_P5.00mm_Wima_Small" H 4200 6500 50  0001 C CNN
 F 3 "" H 4200 6500 50  0001 C CNN
 	1    4200 6500
@@
 F 0 "R14" H 9600 4850 50  0000 R CNN
 F 1 "470K 1/2W" H 9600 4950 50  0000 R CNN
-F 2 "" V 9690 4890 50  0001 C CNN
+F 2 "KiCadCommon:KiCadCommon_R_Axial_0.5W" V 9690 4890 50  0001 C CNN
 F 3 "~" H 9650 4900 50  0001 C CNN
 	1    9650 4900
@@
 F 0 "R15" H 10350 5350 50  0000 R CNN
 F 1 "1.82K 1/2W" H 10350 5450 50  0000 R CNN
-F 2 "KiCadCommon:KiCadCommon_R_Axial_0.5W" V 10440 5390 50  0001 C CNN
+F 2 "KiCadCommon:KiCadCommon_R_Vertical_L9.0mm_D3.2mm_P2.54mm" V 10440 5390 50  0001 C CNN
 F 3 "~" H 10400 5400 50  0001 C CNN
 	1    10400 5400
@@
 F 0 "R16" H 11000 6750 50  0000 R CNN
 F 1 "47K 1/2W" H 11000 6850 50  0000 R CNN
-F 2 "KiCadCommon:KiCadCommon_R_Axial_0.5W" V 11090 6790 50  0001 C CNN
+F 2 "KiCadCommon:KiCadCommon_R_Vertical_L9.0mm_D3.2mm_P2.54mm" V 11090 6790 50  0001 C CNN
 F 3 "~" H 11050 6800 50  0001 C CNN
 	1    11050 6800
@@
 F 0 "R27" V 14600 4150 50  0000 C CNN
 F 1 "1M 1/2W" V 14800 4150 50  0000 C CNN
-F 2 "" V 14740 4140 50  0001 C CNN
+F 2 "KiCadCommon:KiCadCommon_R_Axial_0.5W" V 14740 4140 50  0001 C CNN
 F 3 "~" H 14700 4150 50  0001 C CNN
 	1    14700 4150
@@
 F 0 "R28" H 15468 4954 50  0000 L CNN
 F 1 "100K 1/2W" H 15468 5045 50  0000 L CNN
-F 2 "" V 15440 4990 50  0001 C CNN
+F 2 "KiCadCommon:KiCadCommon_R_Axial_0.5W" V 15440 4990 50  0001 C CNN
 F 3 "~" H 15400 5000 50  0001 C CNN
 	1    15400 5000
@@
 F 0 "R30" H 15950 3750 50  0000 R CNN
 F 1 "220K 1W" H 15950 3850 50  0000 R CNN
-F 2 "" V 16040 3790 50  0001 C CNN
+F 2 "KiCadCommon:KiCadCommon_R_Axial_1W" V 16040 3790 50  0001 C CNN
 F 3 "~" H 16000 3800 50  0001 C CNN
 	1    16000 3800
@@
 F 0 "R29" H 15850 5250 50  0000 R CNN
 F 1 "2.2K 1/2W" H 15850 5350 50  0000 R CNN
-F 2 "" V 15940 5290 50  0001 C CNN
+F 2 "KiCadCommon:KiCadCommon_R_Vertical_L9.0mm_D3.2mm_P2.54mm" V 15940 5290 50  0001 C CNN
 F 3 "~" H 15900 5300 50  0001 C CNN
 	1    15900 5300
@@
 F 0 "R31" V 16250 4150 50  0000 C CNN
 F 1 "1M 1/2W" V 16450 4150 50  0000 C CNN
-F 2 "" V 16390 4140 50  0001 C CNN
+F 2 "KiCadCommon:KiCadCommon_R_Axial_0.5W" V 16390 4140 50  0001 C CNN
 F 3 "~" H 16350 4150 50  0001 C CNN
 	1    16350 4150
@@
 F 0 "R32" H 17150 5050 50  0000 R CNN
 F 1 "1M 1/2W" H 17150 5150 50  0000 R CNN
-F 2 "" V 17240 5090 50  0001 C CNN
+F 2 "KiCadCommon:KiCadCommon_R_Axial_0.5W" V 17240 5090 50  0001 C CNN
 F 3 "~" H 17200 5100 50  0001 C CNN
 	1    17200 5100
@@
 F 0 "R33" V 17350 4350 50  0000 C CNN
 F 1 "1M 1/2W" V 17550 4350 50  0000 C CNN
-F 2 "" V 17490 4340 50  0001 C CNN
+F 2 "KiCadCommon:KiCadCommon_R_Axial_0.5W" V 17490 4340 50  0001 C CNN
 F 3 "~" H 17450 4350 50  0001 C CNN
 	1    17450 4350
@@
 F 0 "R35" H 17750 3750 50  0000 R CNN
 F 1 "100K 1W" H 17750 3850 50  0000 R CNN
-F 2 "" V 17840 3790 50  0001 C CNN
+F 2 "KiCadCommon:KiCadCommon_R_Axial_1W" V 17840 3790 50  0001 C CNN
 F 3 "~" H 17800 3800 50  0001 C CNN
 	1    17800 3800
@@
 F 0 "R34" H 17650 5450 50  0000 R CNN
 F 1 "2.2K 1/2W" H 17650 5550 50  0000 R CNN
-F 2 "" V 17740 5490 50  0001 C CNN
+F 2 "KiCadCommon:KiCadCommon_R_Axial_0.5W" V 17740 5490 50  0001 C CNN
 F 3 "~" H 17700 5500 50  0001 C CNN
 	1    17700 5500
@@
 F 0 "R36" H 18500 4550 50  0000 R CNN
 F 1 "470K 1/2W" H 18500 4650 50  0000 R CNN
-F 2 "" V 18590 4590 50  0001 C CNN
+F 2 "KiCadCommon:KiCadCommon_R_Axial_0.5W" V 18590 4590 50  0001 C CNN
 F 3 "~" H 18550 4600 50  0001 C CNN
 	1    18550 4600
@@
 F 0 "R1" V 3750 6250 50  0000 C CNN
 F 1 "22K 1/2W" V 3950 6250 50  0000 C CNN
-F 2 "" V 3890 6240 50  0001 C CNN
+F 2 "KiCadCommon:KiCadCommon_R_Axial_0.5W" V 3890 6240 50  0001 C CNN
 F 3 "~" H 3850 6250 50  0001 C CNN
 	1    3850 6250
@@
 F 0 "C2" H 3900 5650 50  0000 R CNN
 F 1 ".1uF 50V" H 3900 5500 50  0000 R CNN
-F 2 "" H 4000 5600 50  0001 C CNN
+F 2 "KiCadCommon:KiCadCommon_C_Rect_L7.2mm_W4.5mm_P5.00mm_Wima_Small" H 4000 5600 50  0001 C CNN
 F 3 "" H 4000 5600 50  0001 C CNN
 	1    4000 5600

Commit message: Up
Parts:
- C109, C110, C111: footprint Capacitor_THT:CP_Radial_D13.0mm_P5.00mm -> Capacitor_THT:CP_Radial_D13.0mm_P7.50mm
Changed lines of the file:
@@
 F 0 "C109" H 14100 17950 50  0000 L CNN
 F 1 "22uF" H 14100 17850 50  0000 L CNN
-F 2 "Capacitor_THT:CP_Radial_D13.0mm_P5.00mm" H 14000 17900 50  0001 C CNN
+F 2 "Capacitor_THT:CP_Radial_D13.0mm_P7.50mm" H 14000 17900 50  0001 C CNN
 F 3 "~" H 14000 17900 50  0001 C CNN
 	1    14000 17900
@@
 F 0 "C110" H 15100 17450 50  0000 L CNN
 F 1 "22uF" H 15100 17350 50  0000 L CNN
-F 2 "Capacitor_THT:CP_Radial_D13.0mm_P5.00mm" H 15000 17400 50  0001 C CNN
+F 2 "Capacitor_THT:CP_Radial_D13.0mm_P7.50mm" H 15000 17400 50  0001 C CNN
 F 3 "~" H 15000 17400 50  0001 C CNN
 	1    15000 17400
@@
 F 0 "C111" H 15950 17450 50  0000 L CNN
 F 1 "22uF" H 15950 17350 50  0000 L CNN
-F 2 "Capacitor_THT:CP_Radial_D13.0mm_P5.00mm" H 15850 17400 50  0001 C CNN
+F 2 "Capacitor_THT:CP_Radial_D13.0mm_P7.50mm" H 15850 17400 50  0001 C CNN
 F 3 "~" H 15850 17400 50  0001 C CNN
 	1    15850 17400
