File: Peavey_5150.kicad_pcb (KiCad board)
At the start: 2 copper layers, 280 x 120 mm, 0 parts

Commit message: Thinking...
Parts:
- added C12: 1uF 50V, KiCadCommon:KiCadCommon_CP_Vertical_MP, F.Cu at (265.0, 90.0)
- added C17: 1uF 50V, KiCadCommon:KiCadCommon_CP_Vertical_MP, F.Cu at (250.0, 90.0)
- added C29: 0.0047uF 50v, KiCadCommon:KiCadCommon_CP_Vertical_MP, F.Cu at (236.5, 90.0)
- added C3: 1uF 50V, KiCadCommon:KiCadCommon_CP_Vertical_MP, F.Cu at (235.0, 105.0)
- added J1: INPUT FRONT, KiCadCommon:KiCadCommon_Jack_Horizontal_6.35mm, F.Cu at (345.0, 190.0)
- added J2: INPUT REAR, KiCadCommon:KiCadCommon_Jack_Horizontal_6.35mm, F.Cu at (345.0, 70.0)
- added J3: SEND, KiCadCommon:KiCadCommon_Jack_Horizontal_6.35mm, F.Cu at (190.0, 70.0)
- added J4: RETURN, KiCadCommon:KiCadCommon_Jack_Horizontal_6.35mm, F.Cu at (160.0, 70.0)
- added J5: OUTPUT, KiCadCommon:KiCadCommon_Jack_Horizontal_6.35mm, F.Cu at (130.0, 70.0)
- added J6: FOOTSWITCH, KiCadCommon:KiCadCommon_Jack_Horizontal_6.35mm, F.Cu at (95.0, 70.0)
- added R29: 2.2K 1/2W, KiCadCommon:KiCadCommon_R_Vertical_L9.0mm_D3.2mm_P2.54mm, F.Cu at (250.0, 105.0)
- added R4: 1.82K 1/2W, KiCadCommon:KiCadCommon_R_Vertical_L9.0mm_D3.2mm_P2.54mm, F.Cu at (235.0, 75.0)
- added R50: 3.3K 1/2W, KiCadCommon:KiCadCommon_R_Vertical_L9.0mm_D3.2mm_P2.54mm, F.Cu at (245.0, 75.0)
- added R6: 2.2K 1/2W, KiCadCommon:KiCadCommon_R_Vertical_L9.0mm_D3.2mm_P2.54mm, F.Cu at (263.1, 78.0)
- added V1: , KiCadCommon:KiCadCommon_Tube_Socket_MP, F.Cu at (300.0, 140.0)
- added V2: , KiCadCommon:KiCadCommon_Tube_Socket_MP, F.Cu at (260.0, 140.0)
- added V3: , KiCadCommon:KiCadCommon_Tube_Socket_MP, F.Cu at (190.0, 130.0)
- added V4: , KiCadCommon:KiCadCommon_Tube_Socket_MP, F.Cu at (150.0, 130.0)
- added VR1: 1M LOG, KiCadCommon:KiCadCommon_Potentiometer_Alpha_Single_Horizontal, F.Cu at (305.0, 195.0)
- added VR2: 1M LOG, KiCadCommon:KiCadCommon_Potentiometer_Alpha_Single_Horizontal, F.Cu at (275.0, 195.0)
- added VR3: 250K, KiCadCommon:KiCadCommon_Potentiometer_Alpha_Single_Horizontal, F.Cu at (240.0, 195.0)
- added VR4: 250K, KiCadCommon:KiCadCommon_Potentiometer_Alpha_Single_Horizontal, F.Cu at (210.0, 195.0)
- added VR5: 1M, KiCadCommon:KiCadCommon_Potentiometer_Alpha_Single_Horizontal, F.Cu at (180.0, 195.0)
- added VR6: 25K, KiCadCommon:KiCadCommon_Potentiometer_Alpha_Single_Horizontal, F.Cu at (150.0, 195.0)
- added VR7: 1M LOG, KiCadCommon:KiCadCommon_Potentiometer_Alpha_Single_Horizontal, F.Cu at (115.0, 195.0)
- added VR8: 1M LOG, KiCadCommon:KiCadCommon_Potentiometer_Alpha_Single_Horizontal, F.Cu at (85.0, 195.0)
- added VR9: 1M, KiCadCommon:KiCadCommon_Potentiometer_Alpha_Single_Horizontal, F.Cu at (90.0, 165.0)
Other:
- board size 280 x 120 mm -> 290 x 140 mm

Commit message: Up
Parts:
- moved C12 144.3 mm to (125.0, 125.0)
- moved C17 144.3 mm to (110.0, 125.0)
- moved C29 144.3 mm to (96.5, 125.0)
- moved C3 144.3 mm to (95.0, 140.0)
- moved R29 144.3 mm to (110.0, 140.0)
- moved R4 144.3 mm to (95.0, 110.0)
- moved R50 144.3 mm to (105.0, 110.0)
- moved R6 144.3 mm to (123.1, 113.0)
- moved VR9 125.0 mm to (165.0, 65.0), turned to 90 degrees
- moved J3 30.0 mm to (220.0, 70.0)
- moved J4 30.0 mm to (190.0, 70.0)
Changed lines of the file:
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@@
   )
   (module KiCadCommon:KiCadCommon_CP_Vertical_MP (layer F.Cu)
-    (at 236.5 90)
+    (at 96.5 125)
     (fp_text reference C29 (at 1 -4) (layer F.SilkS)
       (effects (font (size 1 1) (thickness 0.15)))
@@
   )
   (module KiCadCommon:KiCadCommon_R_Vertical_L9.0mm_D3.2mm_P2.54mm (layer F.Cu)
-    (at 235 75)
+    (at 95 110)
     (descr "Resistor, DIN0309 series, Vertical, pin pitch=2.54mm, 0.5W = 1/2W, length*diameter=9*3.2mm^2, http://cdn-reichelt.de/documents/datenblatt/B400/1_4W%23YAG.pdf")
     (tags "Resistor DIN0309 series Vertical pin pitch 2.54mm 0.5W = 1/2W length 9mm diameter 3.2mm")
@@
   )
   (module KiCadCommon:KiCadCommon_R_Vertical_L9.0mm_D3.2mm_P2.54mm (layer F.Cu)
-    (at 263.13 77.95)
+    (at 123.13 112.95)
     (descr "Resistor, DIN0309 series, Vertical, pin pitch=2.54mm, 0.5W = 1/2W, length*diameter=9*3.2mm^2, http://cdn-reichelt.de/documents/datenblatt/B400/1_4W%23YAG.pdf")
     (tags "Resistor DIN0309 series Vertical pin pitch 2.54mm 0.5W = 1/2W length 9mm diameter 3.2mm")
@@
   )
   (module KiCadCommon:KiCadCommon_R_Vertical_L9.0mm_D3.2mm_P2.54mm (layer F.Cu)
-    (at 250 105)
+    (at 110 140)
     (descr "Resistor, DIN0309 series, Vertical, pin pitch=2.54mm, 0.5W = 1/2W, length*diameter=9*3.2mm^2, http://cdn-reichelt.de/documents/datenblatt/B400/1_4W%23YAG.pdf")
     (tags "Resistor DIN0309 series Vertical pin pitch 2.54mm 0.5W = 1/2W length 9mm diameter 3.2mm")
@@
   )
   (module KiCadCommon:KiCadCommon_R_Vertical_L9.0mm_D3.2mm_P2.54mm (layer F.Cu)
-    (at 245 75)
+    (at 105 110)
     (descr "Resistor, DIN0309 series, Vertical, pin pitch=2.54mm, 0.5W = 1/2W, length*diameter=9*3.2mm^2, http://cdn-reichelt.de/documents/datenblatt/B400/1_4W%23YAG.pdf")
     (tags "Resistor DIN0309 series Vertical pin pitch 2.54mm 0.5W = 1/2W length 9mm diameter 3.2mm")
@@
   )
   (module KiCadCommon:KiCadCommon_Potentiometer_Alpha_Single_Horizontal (layer F.Cu)
-    (at 90 165)
+    (at 165 65 90)
     (descr "Potentiometer, horizontal, Alpha Single, http://www.alps.com/prod/info/E/HTML/Potentiometer/RotaryPotentiometers/RK16/RK16_list.html")
     (tags "Potentiometer horizontal Alpha Single")
-    (fp_text reference VR9 (at 0 -15.2) (layer F.SilkS)
-      (effects (font (size 1 1) (thickness 0.15)))
-    )
-    (fp_text value 1M (at 0 5.2) (layer F.Fab)
-      (effects (font (size 1 1) (thickness 0.15)))
-    )
-    (fp_text user %R (at -1.45 -5) (layer F.Fab)
+    (fp_text reference VR9 (at 0 -15.2 90) (layer F.SilkS)
+      (effects (font (size 1 1) (thickness 0.15)))
+    )
+    (fp_text value 1M (at 0 5.2 90) (layer F.Fab)
+      (effects (font (size 1 1) (thickness 0.15)))
+    )
+    (fp_text user %R (at -1.45 -5 90) (layer F.Fab)
       (effects (font (size 1 1) (thickness 0.15)))
     )
@@
     (fp_line (start 4.064 4.191) (end 4.064 -14.224) (layer F.CrtYd) (width 0.05))
     (fp_line (start 4.064 -14.224) (end -6.95 -14.2) (layer F.CrtYd) (width 0.05))
-    (pad 1 thru_hole circle (at 0 0) (size 2.34 2.34) (drill 1.3) (layers *.Cu *.Mask)
-      (net 26 Earth_Protective))
-    (pad 2 thru_hole circle (at 0 -5) (size 2.34 2.34) (drill 1.3) (layers *.Cu *.Mask)
+    (pad 1 thru_hole circle (at 0 0 90) (size 2.34 2.34) (drill 1.3) (layers *.Cu *.Mask)
+      (net 26 Earth_Protective))
+    (pad 2 thru_hole circle (at 0 -5 90) (size 2.34 2.34) (drill 1.3) (layers *.Cu *.Mask)
       (net 27 "Net-(C30-Pad2)"))
-    (pad 3 thru_hole circle (at 0 -10) (size 2.34 2.34) (drill 1.3) (layers *.Cu *.Mask)
+    (pad 3 thru_hole circle (at 0 -10 90) (size 2.34 2.34) (drill 1.3) (layers *.Cu *.Mask)
       (net 35 "Net-(J5-Pad1)"))
     (model ${KIPRJMOD}/KiCadCommonLib/modules/packages3d/KiCadCommon.3dshapes/KiCadCommon_Potentiometer_Alpha_Vertical.stp
@@
   )
   (module KiCadCommon:KiCadCommon_Jack_Horizontal_6.35mm (layer F.Cu)
-    (at 160 70 180)
+    (at 190 70 180)
     (fp_text reference J4 (at 0 -13.1) (layer F.SilkS)
       (effects (font (size 1 1) (thickness 0.15)))
@@
   )
   (module KiCadCommon:KiCadCommon_Jack_Horizontal_6.35mm (layer F.Cu)
-    (at 190 70 180)
+    (at 220 70 180)
     (fp_text reference J3 (at 0 -13.1) (layer F.SilkS)
       (effects (font (size 1 1) (thickness 0.15)))
@@
   )
   (module KiCadCommon:KiCadCommon_CP_Vertical_MP (layer F.Cu)
-    (at 250 90)
+    (at 110 125)
     (fp_text reference C17 (at 1 -4) (layer F.SilkS)
       (effects (font (size 1 1) (thickness 0.15)))
@@
   )
   (module KiCadCommon:KiCadCommon_CP_Vertical_MP (layer F.Cu)
-    (at 265 90)
+    (at 125 125)
     (fp_text reference C12 (at 1 -4) (layer F.SilkS)
       (effects (font (size 1 1) (thickness 0.15)))
@@
   )
   (module KiCadCommon:KiCadCommon_CP_Vertical_MP (layer F.Cu)
-    (at 235 105)
+    (at 95 140)
     (fp_text reference C3 (at 1 -4) (layer F.SilkS)
       (effects (font (size 1 1) (thickness 0.15)))
